File: alice3/kicad/IO/IO.sch (KiCad schematic (older format))
At the start: 22 parts, among them CON1 SD_Card, U1 MiniM4-D40, U2 LEVELCONVERTER, U3 LEVELCONVERTER, U4 LEVELCONVERTER, U5 LEVELCONVERTER, U6 Alice_3_bus, U7 DFROBOT_FTDI_BASIC, U8 LM2937-3.3, X1 MINI_DIN_6

Commit message: begin IO board PCB
Parts:
- removed C1: CP, symbol CP
- added C1: 22µF, Capacitors_ThroughHole:C_Radial_D5_L11_P2, symbol CP1
- C2: value CP1 -> 470µF; footprint (none) -> Capacitors_ThroughHole:C_Radial_D13_L25_P5
- CON1: footprint 10067847-001 -> (none)
- R0, R1, R2, R3, R4, R5, R6: footprint (none) -> Resistors_ThroughHole:Resistor_Horizontal_RM10mm
- U1: footprint (none) -> Housings_DIP:DIP-40_W15.24mm
- U2, U3, U4, U5: footprint (none) -> level converter:LEVELCONV
- X1: footprint mini_din-M_DIN6 -> (none)
Connections:
- net +3V3: now also C1.1
- net GND: now also C1.2
Changed lines of the file:
@@
 F 0 "U1" H 3000 4550 60  0000 C CNN
 F 1 "MiniM4-D40" H 3350 1650 60  0000 C CNN
-F 2 "" H 3200 1600 60  0000 C CNN
+F 2 "Housings_DIP:DIP-40_W15.24mm" H 3200 1600 60  0001 C CNN
 F 3 "" H 3200 1600 60  0000 C CNN
 	1    3350 3100
@@
 F 0 "CON1" H 1350 7450 50  0000 C CNN
 F 1 "SD_Card" H 2600 6350 50  0000 C CNN
-F 2 "10067847-001" H 2200 7250 50  0000 C CNN
+F 2 "" H 2200 7250 50  0001 C CNN
 F 3 "" H 2000 6900 60  0000 C CNN
 	1    2000 6900
@@
 F 0 "R0" V 3330 6300 50  0000 C CNN
 F 1 "68K" V 3250 6300 50  0000 C CNN
-F 2 "" V 3180 6300 30  0000 C CNN
+F 2 "Resistors_ThroughHole:Resistor_Horizontal_RM10mm" V 3180 6300 30  0001 C CNN
 F 3 "" H 3250 6300 30  0000 C CNN
 	1    3250 6300
@@
 F 0 "R1" V 3130 6300 50  0000 C CNN
 F 1 "68K" V 3050 6300 50  0000 C CNN
-F 2 "" V 2980 6300 30  0000 C CNN
+F 2 "Resistors_ThroughHole:Resistor_Horizontal_RM10mm" V 2980 6300 30  0001 C CNN
 F 3 "" H 3050 6300 30  0000 C CNN
 	1    3050 6300
@@
 F 0 "R2" V 3530 6300 50  0000 C CNN
 F 1 "68K" V 3450 6300 50  0000 C CNN
-F 2 "" V 3380 6300 30  0000 C CNN
+F 2 "Resistors_ThroughHole:Resistor_Horizontal_RM10mm" V 3380 6300 30  0001 C CNN
 F 3 "" H 3450 6300 30  0000 C CNN
 	1    3450 6300
@@
 F 0 "R3" V 3730 6300 50  0000 C CNN
 F 1 "68K" V 3650 6300 50  0000 C CNN
-F 2 "" V 3580 6300 30  0000 C CNN
+F 2 "Resistors_ThroughHole:Resistor_Horizontal_RM10mm" V 3580 6300 30  0001 C CNN
 F 3 "" H 3650 6300 30  0000 C CNN
 	1    3650 6300
 	1    0    0    -1
-$EndComp
-$Comp
-L CP C1
-U 1 1 5689AB18
-P 3600 7600
-F 0 "C1" H 3625 7700 50  0000 L CNN
-F 1 "CP" H 3625 7500 50  0000 L CNN
-F 2 "" H 3638 7450 30  0000 C CNN
-F 3 "" H 3600 7600 60  0000 C CNN
-	1    3600 7600
-	0    -1   -1   0
 $EndComp
 $Comp
@@
 F 0 "U6" H 8850 6450 60  0000 C CNN
 F 1 "Alice_3_bus" H 9050 5350 60  0000 C CNN
-F 2 "" H 9000 5950 60  0000 C CNN
+F 2 "" H 9000 5950 60  0001 C CNN
 F 3 "" H 9000 5950 60  0000 C CNN
 	1    9050 5900
@@
 F 0 "U2" H 8700 1750 60  0000 C CNN
 F 1 "LEVELCONVERTER" H 8950 850 60  0000 C CNN
-F 2 "" H 8850 450 60  0000 C CNN
+F 2 "level converter:LEVELCONV" H 8850 450 60  0001 C CNN
 F 3 "" H 8850 450 60  0000 C CNN
 	1    8850 1300
@@
 F 0 "U3" H 8700 2800 60  0000 C CNN
 F 1 "LEVELCONVERTER" H 8950 1900 60  0000 C CNN
-F 2 "" H 8850 1500 60  0000 C CNN
+F 2 "level converter:LEVELCONV" H 8850 1500 60  0001 C CNN
 F 3 "" H 8850 1500 60  0000 C CNN
 	1    8850 2350
@@
 F 0 "U4" H 8700 3850 60  0000 C CNN
 F 1 "LEVELCONVERTER" H 8950 2950 60  0000 C CNN
-F 2 "" H 8850 2550 60  0000 C CNN
+F 2 "level converter:LEVELCONV" H 8850 2550 60  0001 C CNN
 F 3 "" H 8850 2550 60  0000 C CNN
 	1    8850 3400
@@
 F 0 "U5" H 8700 4900 60  0000 C CNN
 F 1 "LEVELCONVERTER" H 8950 4000 60  0000 C CNN
-F 2 "" H 8850 3600 60  0000 C CNN
+F 2 "level converter:LEVELCONV" H 8850 3600 60  0001 C CNN
 F 3 "" H 8850 3600 60  0000 C CNN
 	1    8850 4450
@@
 F 0 "HEART1" H 5100 3450 50  0000 C CNN
 F 1 "LED" H 5250 3300 50  0000 C CNN
-F 2 "" H 5100 3350 60  0000 C CNN
+F 2 "" H 5100 3350 60  0001 C CNN
 F 3 "" H 5100 3350 60  0000 C CNN
 	1    5100 3350
@@
 F 0 "PANIC1" H 1250 4100 50  0000 C CNN
 F 1 "LED" H 1400 3950 50  0000 C CNN
-F 2 "" H 1250 4000 60  0000 C CNN
+F 2 "" H 1250 4000 60  0001 C CNN
 F 3 "" H 1250 4000 60  0000 C CNN
 	1    1250 4000
@@
 F 0 "R5" V 1330 4350 50  0000 C CNN
 F 1 "220" V 1250 4350 50  0000 C CNN
-F 2 "" V 1180 4350 30  0000 C CNN
+F 2 "Resistors_ThroughHole:Resistor_Horizontal_RM10mm" V 1180 4350 30  0001 C CNN
 F 3 "" H 1250 4350 30  0000 C CNN
 	1    1250 4350
@@
 F 0 "R6" V 5180 3700 50  0000 C CNN
 F 1 "220" V 5100 3700 50  0000 C CNN
-F 2 "" V 5030 3700 30  0000 C CNN
+F 2 "Resistors_ThroughHole:Resistor_Horizontal_RM10mm" V 5030 3700 30  0001 C CNN
 F 3 "" H 5100 3700 30  0000 C CNN
 	1    5100 3700
@@
 F 0 "INFO1" H 950 4100 50  0000 C CNN
 F 1 "LED" H 1100 3950 50  0000 C CNN
-F 2 "" H 950 4000 60  0000 C CNN
+F 2 "" H 950 4000 60  0001 C CNN
 F 3 "" H 950 4000 60  0000 C CNN
 	1    950  4000
@@
 F 0 "R4" V 1030 4350 50  0000 C CNN
 F 1 "220" V 950 4350 50  0000 C CNN
-F 2 "" V 880 4350 30  0000 C CNN
+F 2 "Resistors_ThroughHole:Resistor_Horizontal_RM10mm" V 880 4350 30  0001 C CNN
 F 3 "" H 950 4350 30  0000 C CNN
 	1    950  4350
@@
 F 0 "X1" H 3550 1525 50  0000 L BNN
 F 1 "MINI_DIN_6" H 3950 1525 50  0000 L BNN
-F 2 "mini_din-M_DIN6" H 3950 1150 50  0001 C CNN
+F 2 "" H 3950 1150 50  0001 C CNN
 F 3 "" H 3950 1000 60  0000 C CNN
 	1    3950 1000
@@
 F 0 "U7" H 5900 3350 60  0000 C CNN
 F 1 "DFROBOT_FTDI_BASIC" H 6150 2150 60  0000 C CNN
-F 2 "" H 6150 2150 60  0000 C CNN
+F 2 "" H 6150 2150 60  0001 C CNN
 F 3 "" H 6150 2150 60  0000 C CNN
 	1    6150 2750
@@
 F 0 "U8" H 5300 1400 60  0000 C CNN
 F 1 "LM2937-3.3" H 5750 1400 60  0000 C CNN
-F 2 "" H 5550 1200 60  0000 C CNN
+F 2 "" H 5550 1200 60  0001 C CNN
 F 3 "" H 5550 1200 60  0000 C CNN
 	1    5550 1200
@@
 P 6200 1400
 F 0 "C2" H 6225 1500 50  0000 L CNN
-F 1 "CP1" H 6225 1300 50  0000 L CNN
-F 2 "" H 6200 1400 60  0000 C CNN
+F 1 "470µF" H 6225 1300 50  0000 L CNN
+F 2 "Capacitors_ThroughHole:C_Radial_D13_L25_P5" H 6200 1400 60  0001 C CNN
 F 3 "" H 6200 1400 60  0000 C CNN
 	1    6200 1400
@@
 Wire Wire Line
 	6200 1050 6200 1250
+$Comp
+L CP1 C1
+U 1 1 568A9C8C
+P 3600 7600
+F 0 "C1" H 3625 7700 50  0000 L CNN
+F 1 "22µF" H 3625 7500 50  0000 L CNN
+F 2 "Capacitors_ThroughHole:C_Radial_D5_L11_P2" H 3600 7600 60  0001 C CNN
+F 3 "" H 3600 7600 60  0000 C CNN
+	1    3600 7600
+	0    -1   -1   0
+$EndComp
 $EndSCHEMATC

Commit message: more footprints
Parts:
- CON1: footprint (none) -> Connect:SD_Card_Receptacle
- HEART1, INFO1, PANIC1: footprint (none) -> LEDs:LED-5MM
- U6: footprint (none) -> Pin_Headers:Pin_Header_Straight_2x10
- U7: footprint (none) -> ftdi basic breakout:FTDIBASIC
- U8: footprint (none) -> Power_Integrations:TO-220
- X1: footprint (none) -> r_mini_din:Mini_din6
Changed lines of the file:
@@
 F 0 "CON1" H 1350 7450 50  0000 C CNN
 F 1 "SD_Card" H 2600 6350 50  0000 C CNN
-F 2 "" H 2200 7250 50  0001 C CNN
+F 2 "Connect:SD_Card_Receptacle" H 2200 7250 50  0001 C CNN
 F 3 "" H 2000 6900 60  0000 C CNN
 	1    2000 6900
@@
 F 0 "U6" H 8850 6450 60  0000 C CNN
 F 1 "Alice_3_bus" H 9050 5350 60  0000 C CNN
-F 2 "" H 9000 5950 60  0001 C CNN
+F 2 "Pin_Headers:Pin_Header_Straight_2x10" H 9000 5950 60  0001 C CNN
 F 3 "" H 9000 5950 60  0000 C CNN
 	1    9050 5900
@@
 F 0 "HEART1" H 5100 3450 50  0000 C CNN
 F 1 "LED" H 5250 3300 50  0000 C CNN
-F 2 "" H 5100 3350 60  0001 C CNN
+F 2 "LEDs:LED-5MM" H 5250 3300 50  0001 C CNN
 F 3 "" H 5100 3350 60  0000 C CNN
 	1    5100 3350
@@
 F 0 "PANIC1" H 1250 4100 50  0000 C CNN
 F 1 "LED" H 1400 3950 50  0000 C CNN
-F 2 "" H 1250 4000 60  0001 C CNN
+F 2 "LEDs:LED-5MM" H 1400 3950 50  0001 C CNN
 F 3 "" H 1250 4000 60  0000 C CNN
 	1    1250 4000
@@
 F 0 "INFO1" H 950 4100 50  0000 C CNN
 F 1 "LED" H 1100 3950 50  0000 C CNN
-F 2 "" H 950 4000 60  0001 C CNN
+F 2 "LEDs:LED-5MM" H 950 4000 50  0001 C CNN
 F 3 "" H 950 4000 60  0000 C CNN
 	1    950  4000
@@
 F 0 "X1" H 3550 1525 50  0000 L BNN
 F 1 "MINI_DIN_6" H 3950 1525 50  0000 L BNN
-F 2 "" H 3950 1150 50  0001 C CNN
+F 2 "r_mini_din:Mini_din6" H 3950 1150 50  0001 C CNN
 F 3 "" H 3950 1000 60  0000 C CNN
 	1    3950 1000
@@
 F 0 "U7" H 5900 3350 60  0000 C CNN
 F 1 "DFROBOT_FTDI_BASIC" H 6150 2150 60  0000 C CNN
-F 2 "" H 6150 2150 60  0001 C CNN
+F 2 "ftdi basic breakout:FTDIBASIC" H 6150 2150 60  0001 C CNN
 F 3 "" H 6150 2150 60  0000 C CNN
 	1    6150 2750
@@
 F 0 "U8" H 5300 1400 60  0000 C CNN
 F 1 "LM2937-3.3" H 5750 1400 60  0000 C CNN
-F 2 "" H 5550 1200 60  0001 C CNN
+F 2 "Power_Integrations:TO-220" H 5550 1200 60  0001 C CNN
 F 3 "" H 5550 1200 60  0000 C CNN
 	1    5550 1200

Commit message: IO board PCB
Connections:
- net /INT: no longer U5.12 (HV1), U6.3 (/INT)
- net /IORQ: no longer U4.12 (HV1), U6.9 (/IORQ)
- net /M1: no longer U5.7 (HV4), U6.6 (/M1)
- net /RD: no longer U4.11 (HV2), U6.7 (/RD)
- net /RESET: no longer U5.11 (HV2), U6.4 (/RESET)
- net /WAIT: no longer U5.8 (HV3), U6.5 (/WAIT)
- net /WR: no longer U4.8 (HV3), U6.8 (/WR)
- net A7: no longer U4.7 (HV4), U6.19 (A7)
- net D0: no longer U2.12 (HV1), U6.11 (D0)
- net D1: no longer U2.11 (HV2), U6.12 (D1)
- net D2: no longer U2.8 (HV3), U6.13 (D2)
- net D3: no longer U2.7 (HV4), U6.14 (D3)
- net D4: no longer U3.12 (HV1), U6.15 (D4)
- net D5: no longer U3.11 (HV2), U6.16 (D5)
- net D6: no longer U3.8 (HV3), U6.17 (D6)
- net D7: no longer U3.7 (HV4), U6.18 (D7)
- new net /INT.5v: U5.12 (HV1), U6.3 (/INT)
- new net /IORQ.5v: U4.12 (HV1), U6.9 (/IORQ)
- new net /M1.5v: U5.7 (HV4), U6.6 (/M1)
- new net /RD.5v: U4.11 (HV2), U6.7 (/RD)
- new net /RESET.5v: U5.11 (HV2), U6.4 (/RESET)
- new net /WAIT.5v: U5.8 (HV3), U6.5 (/WAIT)
- new net /WR.5v: U4.8 (HV3), U6.8 (/WR)
- new net A7.5v: U4.7 (HV4), U6.19 (A7)
- new net D0.5v: U2.12 (HV1), U6.11 (D0)
- new net D1.5v: U2.11 (HV2), U6.12 (D1)
- new net D2.5v: U2.8 (HV3), U6.13 (D2)
- new net D3.5v: U2.7 (HV4), U6.14 (D3)
- new net D4.5v: U3.12 (HV1), U6.15 (D4)
- new net D5.5v: U3.11 (HV2), U6.16 (D5)
- new net D6.5v: U3.8 (HV3), U6.17 (D6)
- new net D7.5v: U3.7 (HV4), U6.18 (D7)
Changed lines of the file:
@@
 BUS5
 Text Label 9600 1050 0    60   ~ 0
-D0
+D0.5v
 Text Label 9600 1150 0    60   ~ 0
-D1
+D1.5v
 Text Label 9600 1450 0    60   ~ 0
-D2
+D2.5v
 Text Label 9600 1550 0    60   ~ 0
-D3
+D3.5v
 Text Label 9600 2100 0    60   ~ 0
-D4
+D4.5v
 Text Label 9600 2200 0    60   ~ 0
-D5
+D5.5v
 Text Label 9600 2500 0    60   ~ 0
-D6
+D6.5v
 Text Label 9600 2600 0    60   ~ 0
-D7
+D7.5v
 Text Label 9500 3150 0    60   ~ 0
-/IORQ
+/IORQ.5v
 Text Label 9500 3250 0    60   ~ 0
-/RD
+/RD.5v
 Text Label 9500 3550 0    60   ~ 0
-/WR
+/WR.5v
 Text Label 9500 3650 0    60   ~ 0
-A7
+A7.5v
 Text Label 9500 4200 0    60   ~ 0
-/INT
+/INT.5v
 Text Label 9500 4300 0    60   ~ 0
-/RESET
+/RESET.5v
 Text Label 9550 4600 0    60   ~ 0
-/WAIT
+/WAIT.5v
 Text Label 9550 4700 0    60   ~ 0
-/M1
+/M1.5v
 Entry Wire Line
 	9700 5450 9800 5550
@@
 BUS5
 Text Label 8400 5650 0    60   ~ 0
-/INT
+/INT.5v
 Text Label 8400 5750 0    60   ~ 0
-/RESET
+/RESET.5v
 Text Label 8400 5850 0    60   ~ 0
-/WAIT
+/WAIT.5v
 Text Label 8400 5950 0    60   ~ 0
-/M1
+/M1.5v
 Text Label 8400 6050 0    60   ~ 0
-/RD
+/RD.5v
 Text Label 8400 6150 0    60   ~ 0
-/WR
+/WR.5v
 Text Label 8400 6250 0    60   ~ 0
-/IORQ
+/IORQ.5v
 Text Label 9550 5450 0    60   ~ 0
-D0
+D0.5v
 Text Label 9550 5550 0    60   ~ 0
-D1
+D1.5v
 Text Label 9550 5650 0    60   ~ 0
-D2
+D2.5v
 Text Label 9550 5750 0    60   ~ 0
-D3
+D3.5v
 Text Label 9550 5850 0    60   ~ 0
-D4
+D4.5v
 Text Label 9550 5950 0    60   ~ 0
-D5
+D5.5v
 Text Label 9550 6050 0    60   ~ 0
-D6
+D6.5v
 Text Label 9550 6150 0    60   ~ 0
-D7
+D7.5v
 Text Label 9550 6250 0    60   ~ 0
-A7
+A7.5v
 $Comp
 L +5V #PWR026
