File: alice3/kicad/MOBO/VIDEO.sch (KiCad schematic (older format))
At the start: 17 parts, among them SW1 RESET, U1 Propeller_P8X32A-D40, U2 VGA_daughter_board, U3 24LC256, U4 Propeller_Plug, U5 LM2937-3.3, U6 74HC4050, U7 74HC4050, U8 Alice_3_bus, Y1 5 MHz

Commit message: Clean up VIDEO.
Parts:
- removed U6, U7: 74HC4050, Housings_DIP:DIP-16_W7.62mm, symbol 74HC4050
- removed U8: Alice_3_bus, Pin_Headers:Pin_Header_Straight_2x10, symbol Alice_3_bus
Connections:
- net labels added: KBD_CLK, KBD_DATA
- wire segments 138 -> 102
- no-connect marks 16 -> 8
Other:
- moved on the sheet: U2

Commit message: More VIDEO cleanup.
Parts:
- added C?: 0.1 µF, symbol C
Connections:
- net +3V3: now also C?.1
- net /IORQ: now also U1.2 (P1); no longer U1.33 (P24)
- net /WR: now also U1.3 (P2); no longer U1.34 (P25)
- net A7: now also U1.5 (P4); no longer U1.35 (P26)
- net GND: now also C?.2
- net /RD: now reaches U1.4 (P3)
- no-connect marks 8 -> 9
Other:
- moved on the sheet: D2, R4
Changed lines of the file:
@@
 L LED D2
 U 1 1 56821EAA
-P 5900 2600
-F 0 "D2" H 5900 2700 50  0000 C CNN
-F 1 "DEBUG" H 5900 2500 50  0000 C CNN
-F 2 "LEDs:LED-5MM" H 5900 2600 50  0001 C CNN
-F 3 "" H 5900 2600 50  0000 C CNN
-	1    5900 2600
+P 5700 2600
+F 0 "D2" H 5700 2700 50  0000 C CNN
+F 1 "DEBUG" H 5700 2500 50  0000 C CNN
+F 2 "LEDs:LED-5MM" H 5700 2600 50  0001 C CNN
+F 3 "" H 5700 2600 50  0000 C CNN
+	1    5700 2600
 	1    0    0    -1
 $EndComp
@@
 L R R4
 U 1 1 56821F00
-P 5700 2850
-F 0 "R4" V 5780 2850 50  0000 C CNN
-F 1 "100" V 5700 2850 50  0000 C CNN
-F 2 "Resistors_ThroughHole:Resistor_Horizontal_RM10mm" V 5630 2850 50  0001 C CNN
-F 3 "" H 5700 2850 50  0000 C CNN
-	1    5700 2850
+P 5500 2850
+F 0 "R4" V 5580 2850 50  0000 C CNN
+F 1 "100" V 5500 2850 50  0000 C CNN
+F 2 "Resistors_ThroughHole:Resistor_Horizontal_RM10mm" V 5430 2850 50  0001 C CNN
+F 3 "" H 5500 2850 50  0000 C CNN
+	1    5500 2850
 	1    0    0    -1
 $EndComp
@@
 L GND #PWR016
 U 1 1 56821F3F
-P 5700 3100
-F 0 "#PWR016" H 5700 2850 50  0001 C CNN
-F 1 "GND" H 5700 2950 50  0000 C CNN
-F 2 "" H 5700 3100 50  0000 C CNN
-F 3 "" H 5700 3100 50  0000 C CNN
-	1    5700 3100
-	1    0    0    -1
-$EndComp
-NoConn ~ 6200 2700
-NoConn ~ 6200 2800
-NoConn ~ 6200 2900
-NoConn ~ 6200 3000
-NoConn ~ 6200 3100
-NoConn ~ 6200 3200
+P 5500 3100
+F 0 "#PWR016" H 5500 2850 50  0001 C CNN
+F 1 "GND" H 5500 2950 50  0000 C CNN
+F 2 "" H 5500 3100 50  0000 C CNN
+F 3 "" H 5500 3100 50  0000 C CNN
+	1    5500 3100
+	1    0    0    -1
+$EndComp
 NoConn ~ 6200 3300
-Entry Wire Line
-	7500 2600 7600 2700
-Entry Wire Line
-	7500 2700 7600 2800
-Entry Wire Line
-	7500 2800 7600 2900
-Entry Wire Line
-	7500 2900 7600 3000
-Entry Wire Line
-	7500 3000 7600 3100
-Entry Wire Line
-	7500 3100 7600 3200
-Entry Wire Line
-	7500 3200 7600 3300
-Entry Wire Line
-	7500 3300 7600 3400
-Entry Wire Line
-	7500 3500 7600 3600
-Entry Wire Line
-	7500 3600 7600 3700
-Entry Wire Line
-	7500 3700 7600 3800
-Text GLabel 7700 2600 2    60   Input ~ 0
-BUS3.3
-Text Label 7500 2600 2    60   ~ 0
-D0
-Text Label 7500 2700 2    60   ~ 0
-D1
-Text Label 7500 2800 2    60   ~ 0
-D2
-Text Label 7500 2900 2    60   ~ 0
-D3
-Text Label 7500 3000 2    60   ~ 0
-D4
-Text Label 7500 3100 2    60   ~ 0
-D5
-Text Label 7500 3200 2    60   ~ 0
-D6
-Text Label 7500 3300 2    60   ~ 0
-D7
-Text Label 7400 3500 0    60   ~ 0
-/IORQ
-Text Label 7400 3600 0    60   ~ 0
-/WR
-Text Label 7400 3700 0    60   ~ 0
-A7
 NoConn ~ 7400 3800
 $Comp
 L GND #PWR021
 U 1 1 56826035
-P 7600 2400
-F 0 "#PWR021" H 7600 2150 50  0001 C CNN
-F 1 "GND" H 7600 2250 50  0000 C CNN
-F 2 "" H 7600 2400 50  0000 C CNN
-F 3 "" H 7600 2400 50  0000 C CNN
-	1    7600 2400
+P 7450 2400
+F 0 "#PWR021" H 7450 2150 50  0001 C CNN
+F 1 "GND" H 7450 2250 50  0000 C CNN
+F 2 "" H 7450 2400 50  0000 C CNN
+F 3 "" H 7450 2400 50  0000 C CNN
+	1    7450 2400
 	1    0    0    -1
 $EndComp
@@
 	6200 4400 6100 4400
 Wire Wire Line
-	6100 4400 6100 4500
-Wire Wire Line
-	6100 4500 6100 4700
+	6100 4400 6100 4700
 Wire Wire Line
 	6200 4500 6100 4500
@@
 	6100 2400 6200 2400
 Wire Wire Line
-	6100 2100 6100 2300
-Wire Wire Line
-	6100 2300 6100 2400
+	6100 2100 6100 2400
 Wire Wire Line
 	6200 2300 6100 2300
@@
 	7500 4600 7750 4600
 Wire Wire Line
-	7400 2400 7600 2400
+	7400 2400 7450 2400
 Wire Wire Line
 	7900 1800 7900 1700
 Wire Wire Line
-	7400 2300 7850 2300
-Wire Wire Line
-	7850 2300 7900 2300
-Wire Wire Line
-	7900 2300 8000 2300
+	7400 2300 8000 2300
 Wire Wire Line
 	7900 2300 7900 2100
@@
 	8400 4000 8350 4000
 Wire Wire Line
-	8350 4000 8350 4100
-Wire Wire Line
-	8350 4100 8350 4200
-Wire Wire Line
-	8350 4200 8350 4300
-Wire Wire Line
-	8350 4300 8350 4400
+	8350 4000 8350 4400
 Wire Wire Line
 	8400 4100 8350 4100
@@
 	9450 4700 8100 4700
 Wire Wire Line
-	8100 4700 8100 4000
-Wire Wire Line
-	8100 4000 8100 3950
+	8100 4700 8100 3950
 Wire Wire Line
 	8100 4000 7400 4000
@@
 	9250 2300 9250 2700
 Wire Wire Line
-	8600 2300 8650 2300
-Wire Wire Line
-	8650 2300 9250 2300
+	8600 2300 9250 2300
 Wire Wire Line
 	8650 2300 8650 2400
 Connection ~ 8650 2300
 Wire Wire Line
-	3900 2800 3900 2850
-Wire Wire Line
-	3900 2850 3900 3000
+	3900 2800 3900 3000
 Wire Wire Line
 	3400 2400 3300 2400
@@
 	3300 2400 3300 2300
 Wire Wire Line
-	4400 2400 4500 2400
-Wire Wire Line
-	4500 2400 4800 2400
-Wire Wire Line
-	4500 2300 4500 2400
-Wire Wire Line
-	4500 2400 4500 2500
+	4400 2400 4800 2400
+Wire Wire Line
+	4500 2300 4500 2500
 Connection ~ 4500 2400
 Wire Wire Line
 	4500 2800 4500 2850
 Wire Wire Line
-	3900 2850 4500 2850
-Wire Wire Line
-	4500 2850 5300 2850
+	3900 2850 5300 2850
 Connection ~ 3900 2850
 Wire Wire Line
@@
 Connection ~ 4500 2850
 Wire Wire Line
-	5700 2700 5700 2600
-Wire Wire Line
-	6100 2600 6200 2600
-Wire Wire Line
-	5700 3100 5700 3000
-Wire Bus Line
-	7600 2600 7600 2700
-Wire Bus Line
-	7600 2700 7600 2800
-Wire Bus Line
-	7600 2800 7600 2900
-Wire Bus Line
-	7600 2900 7600 3000
-Wire Bus Line
-	7600 3000 7600 3100
-Wire Bus Line
-	7600 3100 7600 3200
-Wire Bus Line
-	7600 3200 7600 3300
-Wire Bus Line
-	7600 3300 7600 3400
-Wire Bus Line
-	7600 3400 7600 3600
-Wire Bus Line
-	7600 3600 7600 3700
-Wire Bus Line
-	7600 3700 7600 3800
+	5500 2700 5500 2600
+Wire Wire Line
+	5900 2600 6200 2600
+Wire Wire Line
+	5500 3100 5500 3000
 Wire Wire Line
 	7400 2600 7500 2600
@@
 Wire Wire Line
 	7400 3300 7500 3300
-Wire Wire Line
-	7400 3500 7500 3500
-Wire Wire Line
-	7400 3600 7500 3600
-Wire Wire Line
-	7400 3700 7500 3700
-Wire Bus Line
-	7600 2600 7700 2600
 Wire Wire Line
 	8300 2800 8300 2500
@@
 Wire Wire Line
 	5500 4600 5550 4600
+NoConn ~ 5500 4300
+NoConn ~ 5500 4400
+Text GLabel 7500 2600 2    60   BiDi ~ 0
+D0
+Text GLabel 7500 2700 2    60   BiDi ~ 0
+D1
+Text GLabel 7500 2800 2    60   BiDi ~ 0
+D2
+Text GLabel 7500 2900 2    60   BiDi ~ 0
+D3
+Text GLabel 7500 3000 2    60   BiDi ~ 0
+D4
+Text GLabel 7500 3100 2    60   BiDi ~ 0
+D5
+Text GLabel 7500 3200 2    60   BiDi ~ 0
+D6
+Text GLabel 7500 3300 2    60   BiDi ~ 0
+D7
+NoConn ~ 7400 3500
+NoConn ~ 7400 3600
+NoConn ~ 7400 3700
+Text GLabel 6200 2700 0    60   Input ~ 0
+/IORQ
+Text GLabel 6200 2800 0    60   Input ~ 0
+/WR
+Text GLabel 6200 3000 0    60   Input ~ 0
+A7
+NoConn ~ 6200 3100
+NoConn ~ 6200 3200
+Text GLabel 6200 2900 0    60   Input ~ 0
+/RD
+$Comp
+L C C?
+U 1 1 568DD525
+P 5800 1950
+F 0 "C?" H 5825 2050 50  0000 L CNN
+F 1 "0.1 µF" H 5825 1850 50  0000 L CNN
+F 2 "" H 5838 1800 50  0000 C CNN
+F 3 "" H 5800 1950 50  0000 C CNN
+	1    5800 1950
+	1    0    0    -1
+$EndComp
+$Comp
+L GND #PWR?
+U 1 1 568DD571
+P 5800 2200
+F 0 "#PWR?" H 5800 1950 50  0001 C CNN
+F 1 "GND" H 5800 2050 50  0000 C CNN
+F 2 "" H 5800 2200 50  0000 C CNN
+F 3 "" H 5800 2200 50  0000 C CNN
+	1    5800 2200
+	1    0    0    -1
+$EndComp
+$Comp
+L +3.3V #PWR?
+U 1 1 568DD5A9
+P 5800 1700
+F 0 "#PWR?" H 5800 1550 50  0001 C CNN
+F 1 "+3.3V" H 5800 1840 50  0000 C CNN
+F 2 "" H 5800 1700 50  0000 C CNN
+F 3 "" H 5800 1700 50  0000 C CNN
+	1    5800 1700
+	1    0    0    -1
+$EndComp
+Wire Wire Line
+	5800 1700 5800 1800
+Wire Wire Line
+	5800 2100 5800 2200
 $EndSCHEMATC
