File: alice3/kicad/MOBO/CPU.sch (KiCad schematic (older format))
At the start: 1 part

Commit message: Add SRAM and EEPROM.
Parts:
- added C3: 2.2 µF, symbol CP
- added R7: 1k, symbol R
- added SW2: RESET, symbol SW_PUSH
- added U?: KM681000BLP-7, symbol KM681000BLP-7
- added U?: 28F512, symbol 28F512
- gave numbers to parts that had none: 1
Connections:
- net labels added: /INT_5v, /RESET_5v
- wire segments 38 -> 45
Changed lines of the file:
@@
 LIBS:vga_daughter_board
 LIBS:Zilog
+LIBS:km681000blp-7
+LIBS:28f512
 LIBS:MOBO-cache
 EELAYER 25 0
@@
 $EndDescr
 $Comp
-L Z80CPU U?
+L Z80CPU U6
 U 1 1 568DDED4
 P 5300 3600
-F 0 "U?" H 4750 5000 50  0000 L CNN
+F 0 "U6" H 4750 5000 50  0000 L CNN
 F 1 "Z80CPU" H 5550 5000 50  0000 L CNN
 F 2 "" H 5300 4000 50  0000 C CNN
@@
 $EndComp
 $Comp
-L GND #PWR?
+L GND #PWR52
 U 1 1 568DE0B3
 P 5300 5200
-F 0 "#PWR?" H 5300 4950 50  0001 C CNN
+F 0 "#PWR52" H 5300 4950 50  0001 C CNN
 F 1 "GND" H 5300 5050 50  0000 C CNN
 F 2 "" H 5300 5200 50  0000 C CNN
@@
 $EndComp
 $Comp
-L +5V #PWR?
+L +5V #PWR51
 U 1 1 568DE0CB
 P 5300 2000
-F 0 "#PWR?" H 5300 1850 50  0001 C CNN
+F 0 "#PWR51" H 5300 1850 50  0001 C CNN
 F 1 "+5V" H 5300 2140 50  0000 C CNN
 F 2 "" H 5300 2000 50  0000 C CNN
@@
 D0_5v
 $Comp
-L +5V #PWR?
+L +5V #PWR50
 U 1 1 568DE771
 P 4400 2950
-F 0 "#PWR?" H 4400 2800 50  0001 C CNN
+F 0 "#PWR50" H 4400 2800 50  0001 C CNN
 F 1 "+5V" H 4400 3090 50  0000 C CNN
 F 2 "" H 4400 2950 50  0000 C CNN
@@
 $EndComp
 Wire Wire Line
-	4400 2950 4400 3000
-Wire Wire Line
-	4400 3000 4400 3100
-Wire Wire Line
-	4400 3100 4400 3600
-Wire Wire Line
-	4400 3100 4600 3100
-Wire Wire Line
-	4600 3000 4400 3000
+	4400 2950 4400 3600
+Wire Wire Line
+	4400 3000 4600 3000
 Connection ~ 4400 3000
 Text GLabel 4500 4100 0    60   Output ~ 0
@@
 Wire Wire Line
 	4500 4800 4600 4800
-Connection ~ 4400 3100
+Text GLabel 4300 3100 0    60   Input ~ 0
+/INT_5v
+Wire Wire Line
+	4600 3100 4300 3100
+Text GLabel 3000 2400 0    60   Input ~ 0
+/RESET_5v
+$Comp
+L CP C3
+U 1 1 568DF3E6
+P 3600 2650
+F 0 "C3" H 3625 2750 50  0000 L CNN
+F 1 "2.2 µF" H 3625 2550 50  0000 L CNN
+F 2 "" H 3638 2500 50  0000 C CNN
+F 3 "" H 3600 2650 50  0000 C CNN
+	1    3600 2650
+	1    0    0    -1
+$EndComp
+$Comp
+L R R7
+U 1 1 568DF407
+P 4200 2150
+F 0 "R7" V 4280 2150 50  0000 C CNN
+F 1 "1k" V 4200 2150 50  0000 C CNN
+F 2 "" V 4130 2150 50  0000 C CNN
+F 3 "" H 4200 2150 50  0000 C CNN
+	1    4200 2150
+	1    0    0    -1
+$EndComp
+$Comp
+L SW_PUSH SW2
+U 1 1 568DF428
+P 3200 2800
+F 0 "SW2" H 3350 2910 50  0000 C CNN
+F 1 "RESET" H 3200 2720 50  0000 C CNN
+F 2 "" H 3200 2800 50  0000 C CNN
+F 3 "" H 3200 2800 50  0000 C CNN
+	1    3200 2800
+	0    -1   -1   0
+$EndComp
+$Comp
+L +5V #PWR49
+U 1 1 568DF44C
+P 4200 1950
+F 0 "#PWR49" H 4200 1800 50  0001 C CNN
+F 1 "+5V" H 4200 2090 50  0000 C CNN
+F 2 "" H 4200 1950 50  0000 C CNN
+F 3 "" H 4200 1950 50  0000 C CNN
+	1    4200 1950
+	1    0    0    -1
+$EndComp
+$Comp
+L GND #PWR48
+U 1 1 568DF463
+P 3400 3200
+F 0 "#PWR48" H 3400 2950 50  0001 C CNN
+F 1 "GND" H 3400 3050 50  0000 C CNN
+F 2 "" H 3400 3200 50  0000 C CNN
+F 3 "" H 3400 3200 50  0000 C CNN
+	1    3400 3200
+	1    0    0    -1
+$EndComp
+Wire Wire Line
+	3200 2500 3200 2400
+Connection ~ 3200 2400
+Wire Wire Line
+	3600 2500 3600 2400
+Connection ~ 3600 2400
+Wire Wire Line
+	4200 2000 4200 1950
+Wire Wire Line
+	4600 2400 3000 2400
+Wire Wire Line
+	4200 2300 4200 2400
+Connection ~ 4200 2400
+Wire Wire Line
+	3600 2800 3600 3150
+Wire Wire Line
+	3600 3150 3200 3150
+Wire Wire Line
+	3200 3150 3200 3100
+Wire Wire Line
+	3400 3200 3400 3150
+Connection ~ 3400 3150
+$Comp
+L KM681000BLP-7 U?
+U 1 1 568E02F3
+P 8200 3350
+F 0 "U?" H 8200 4550 50  0000 C CNN
+F 1 "KM681000BLP-7" H 8270 2150 50  0000 C CNN
+F 2 "" H 8200 3350 50  0000 C CNN
+F 3 "" H 8200 3350 50  0000 C CNN
+	1    8200 3350
+	1    0    0    -1
+$EndComp
+$Comp
+L 28F512 U?
+U 1 1 568E0849
+P 2250 5000
+F 0 "U?" H 2250 6200 50  0000 C CNN
+F 1 "28F512" H 2250 3800 50  0000 C CNN
+F 2 "" H 2250 5000 50  0000 C CNN
+F 3 "" H 2250 5000 50  0000 C CNN
+	1    2250 5000
+	1    0    0    -1
+$EndComp
 $EndSCHEMATC

Commit message: first draft completed integration
Parts:
- added U13: 74LS04, symbol 74LS04
- added U14, U17: 74LS32, symbol 74LS32
- added U16: 74LS74, symbol 74LS74
- gave numbers to parts that had none: 2
- renumbered C3 to C4, R7 to R12, U6 to U15
Connections:
- net labels added: CLK
- wire segments 45 -> 80
- no-connect marks 3 -> 4
Other:
- moved on the sheet: C4, R12, SW2, U15, U18

Commit message: remove some unused lines, attach +5 to Vcc on 74xx
Changed lines of the file:
@@
 $EndComp
 $Comp
-L GND #PWR048
+L GND #PWR044
 U 1 1 568DE0B3
 P 3850 7200
-F 0 "#PWR048" H 3850 6950 50  0001 C CNN
+F 0 "#PWR044" H 3850 6950 50  0001 C CNN
 F 1 "GND" H 3850 7050 50  0000 C CNN
 F 2 "" H 3850 7200 50  0000 C CNN
@@
 $EndComp
 $Comp
-L +5V #PWR049
+L +5V #PWR045
 U 1 1 568DE0CB
 P 3850 4000
-F 0 "#PWR049" H 3850 3850 50  0001 C CNN
+F 0 "#PWR045" H 3850 3850 50  0001 C CNN
 F 1 "+5V" H 3850 4140 50  0000 C CNN
 F 2 "" H 3850 4000 50  0000 C CNN
@@
 D0_5v
 $Comp
-L +5V #PWR050
+L +5V #PWR046
 U 1 1 568DE771
 P 2950 4950
-F 0 "#PWR050" H 2950 4800 50  0001 C CNN
+F 0 "#PWR046" H 2950 4800 50  0001 C CNN
 F 1 "+5V" H 2950 5090 50  0000 C CNN
 F 2 "" H 2950 4950 50  0000 C CNN
@@
 $EndComp
 $Comp
-L +5V #PWR051
+L +5V #PWR047
 U 1 1 568DF44C
 P 2750 3950
-F 0 "#PWR051" H 2750 3800 50  0001 C CNN
+F 0 "#PWR047" H 2750 3800 50  0001 C CNN
 F 1 "+5V" H 2750 4090 50  0000 C CNN
 F 2 "" H 2750 3950 50  0000 C CNN
@@
 $EndComp
 $Comp
-L GND #PWR052
+L GND #PWR048
 U 1 1 568DF463
 P 1950 5200
-F 0 "#PWR052" H 1950 4950 50  0001 C CNN
+F 0 "#PWR048" H 1950 4950 50  0001 C CNN
 F 1 "GND" H 1950 5050 50  0000 C CNN
 F 2 "" H 1950 5200 50  0000 C CNN
@@
 $EndComp
 $Comp
-L GND #PWR053
+L GND #PWR049
 U 1 1 568E12CE
 P 4950 950
-F 0 "#PWR053" H 4950 700 50  0001 C CNN
+F 0 "#PWR049" H 4950 700 50  0001 C CNN
 F 1 "GND" H 4950 800 50  0000 C CNN
 F 2 "" H 4950 950 60  0000 C CNN
@@
 $EndComp
 $Comp
-L +5V #PWR054
+L +5V #PWR050
 U 1 1 568E1300
 P 5100 1700
-F 0 "#PWR054" H 5100 1550 50  0001 C CNN
+F 0 "#PWR050" H 5100 1550 50  0001 C CNN
 F 1 "+5V" H 5100 1840 50  0000 C CNN
 F 2 "" H 5100 1700 60  0000 C CNN
@@
 A0_5v
 $Comp
-L +5V #PWR055
+L +5V #PWR051
 U 1 1 568E215B
 P 6900 2950
-F 0 "#PWR055" H 6900 2800 50  0001 C CNN
+F 0 "#PWR051" H 6900 2800 50  0001 C CNN
 F 1 "+5V" H 6900 3090 50  0000 C CNN
 F 2 "" H 6900 2950 60  0000 C CNN
@@
 D0_5v
 $Comp
-L +5V #PWR056
+L +5V #PWR052
 U 1 1 568E25EC
 P 9150 2000
-F 0 "#PWR056" H 9150 1850 50  0001 C CNN
+F 0 "#PWR052" H 9150 1850 50  0001 C CNN
 F 1 "+5V" H 9150 2140 50  0000 C CNN
 F 2 "" H 9150 2000 60  0000 C CNN
@@
 	9150 2000 9100 2000
 $Comp
-L GND #PWR057
+L GND #PWR053
 U 1 1 568E2687
 P 9150 2100
-F 0 "#PWR057" H 9150 1850 50  0001 C CNN
+F 0 "#PWR053" H 9150 1850 50  0001 C CNN
 F 1 "GND" H 9150 1950 50  0000 C CNN
 F 2 "" H 9150 2100 60  0000 C CNN
@@
 /RD_5v
 $Comp
-L +5V #PWR058
+L +5V #PWR054
 U 1 1 568E2984
 P 9650 5050
-F 0 "#PWR058" H 9650 4900 50  0001 C CNN
+F 0 "#PWR054" H 9650 4900 50  0001 C CNN
 F 1 "+5V" H 9650 5190 50  0000 C CNN
 F 2 "" H 9650 5050 60  0000 C CNN
@@
 $EndComp
 $Comp
-L GND #PWR059
+L GND #PWR055
 U 1 1 568E29B9
 P 9650 5350
-F 0 "#PWR059" H 9650 5100 50  0001 C CNN
+F 0 "#PWR055" H 9650 5100 50  0001 C CNN
 F 1 "GND" H 9650 5200 50  0000 C CNN
 F 2 "" H 9650 5350 60  0000 C CNN
@@
 /WR_5v
 $Comp
-L GND #PWR060
+L GND #PWR056
 U 1 1 568E2BE1
 P 6700 2650
-F 0 "#PWR060" H 6700 2400 50  0001 C CNN
+F 0 "#PWR056" H 6700 2400 50  0001 C CNN
 F 1 "GND" H 6700 2500 50  0000 C CNN
 F 2 "" H 6700 2650 60  0000 C CNN
@@
 Wire Wire Line
 	2550 4700 3150 4700
+$Comp
+L +5V #PWR057
+U 1 1 568E2E29
+P 4450 1050
+F 0 "#PWR057" H 4450 900 50  0001 C CNN
+F 1 "+5V" H 4450 1190 50  0000 C CNN
+F 2 "" H 4450 1050 60  0000 C CNN
+F 3 "" H 4450 1050 60  0000 C CNN
+	1    4450 1050
+	1    0    0    -1
+$EndComp
 $EndSCHEMATC

Commit message: Sync schematic with breadboard.
Parts:
- removed C4: 2.2 µF, symbol CP
- removed SW2: RESET, symbol SW_PUSH
- removed U13: 74LS04, symbol 74LS04
- removed U14, U17: 74LS32, symbol 74LS32
- removed U16: 74LS74, symbol 74LS74
- removed U19: 28F512, symbol 28F512
- added R10, R9: 1k, symbol R
- added R11, R13, R14, R15, R16: 10k, symbol R
- R12: value 1k -> 10k
- renumbered U15 to U8, U18 to U9
Connections:
- net labels added: /BUSACK, /BUSRQ, /IORQ, /MREQ, /RD, /WR, /Z80_RESET, A0, A1, A10, A11, A12, A13, A14, A15, A2, A3, A4, A5, A6, A7, A8, A9, D0, D1, D2, D3, D4, D5, D6, D7
- net labels removed: /BUSACK_5v, /BUSRQ_5v, /INT_5v, /IORQ_5v, /MREQ_5v, /RD_5v, /RESET_5v, /WR_5v, A0_5v, A10_5v, A11_5v, A12_5v, A13_5v, A14_5v, A15_5v, A1_5v, A2_5v, A3_5v, A4_5v, A5_5v, A6_5v, A7_5v, A8_5v, A9_5v, D0_5v, D1_5v, D2_5v, D3_5v, D4_5v, D5_5v, D6_5v, D7_5v
- wire segments 80 -> 59
- no-connect marks 4 -> 3
Other:
- moved on the sheet: U8, U9

Commit message: Start PCB.
Parts:
- R10, R11, R12, R13, R14, R15, R16, R9: footprint (none) -> Resistors_ThroughHole:Resistor_Horizontal_RM10mm
- U8: footprint (none) -> Housings_DIP:DIP-40_W15.24mm
- U9: footprint (none) -> Housings_DIP:DIP-32_W15.24mm
Connections:
- net /HALT: now reaches U8.18 (~HALT~)
- no-connect marks 3 -> 2
Changed lines of the file:
@@
 Wire Wire Line
 	3300 3800 3400 3800
-NoConn ~ 3400 3100
 NoConn ~ 3400 2900
 Wire Wire Line
@@
 F 0 "U9" H 7450 4450 50  0000 C CNN
 F 1 "KM681000BLP-7" H 7520 2050 50  0000 C CNN
-F 2 "" H 7450 3250 50  0000 C CNN
+F 2 "Housings_DIP:DIP-32_W15.24mm" H 7450 3250 50  0001 C CNN
 F 3 "" H 7450 3250 50  0000 C CNN
 	1    7450 3250
@@
 F 0 "R9" V 2280 2200 50  0000 C CNN
 F 1 "1k" V 2200 2200 50  0000 C CNN
-F 2 "" V 2130 2200 50  0000 C CNN
+F 2 "Resistors_ThroughHole:Resistor_Horizontal_RM10mm" V 2130 2200 50  0001 C CNN
 F 3 "" H 2200 2200 50  0000 C CNN
 	1    2200 2200
@@
 F 0 "U8" H 3550 4400 50  0000 L CNN
 F 1 "Z80CPU" H 4350 4400 50  0000 L CNN
-F 2 "" H 4100 3400 50  0000 C CNN
+F 2 "Housings_DIP:DIP-40_W15.24mm" H 4100 3400 50  0001 C CNN
 F 3 "" H 4100 3400 50  0000 C CNN
 	1    4100 3000
@@
 F 0 "R11" V 6130 4900 50  0000 C CNN
 F 1 "10k" V 6050 4900 50  0000 C CNN
-F 2 "" V 5980 4900 50  0000 C CNN
+F 2 "Resistors_ThroughHole:Resistor_Horizontal_RM10mm" V 5980 4900 50  0001 C CNN
 F 3 "" H 6050 4900 50  0000 C CNN
 	1    6050 4900
@@
 F 0 "R12" V 6130 5100 50  0000 C CNN
 F 1 "10k" V 6050 5100 50  0000 C CNN
-F 2 "" V 5980 5100 50  0000 C CNN
+F 2 "Resistors_ThroughHole:Resistor_Horizontal_RM10mm" V 5980 5100 50  0001 C CNN
 F 3 "" H 6050 5100 50  0000 C CNN
 	1    6050 5100
@@
 F 0 "R13" V 6130 5300 50  0000 C CNN
 F 1 "10k" V 6050 5300 50  0000 C CNN
-F 2 "" V 5980 5300 50  0000 C CNN
+F 2 "Resistors_ThroughHole:Resistor_Horizontal_RM10mm" V 5980 5300 50  0001 C CNN
 F 3 "" H 6050 5300 50  0000 C CNN
 	1    6050 5300
@@
 F 0 "R14" V 6130 5500 50  0000 C CNN
 F 1 "10k" V 6050 5500 50  0000 C CNN
-F 2 "" V 5980 5500 50  0000 C CNN
+F 2 "Resistors_ThroughHole:Resistor_Horizontal_RM10mm" V 5980 5500 50  0001 C CNN
 F 3 "" H 6050 5500 50  0000 C CNN
 	1    6050 5500
@@
 F 0 "R15" V 6130 5700 50  0000 C CNN
 F 1 "10k" V 6050 5700 50  0000 C CNN
-F 2 "" V 5980 5700 50  0000 C CNN
+F 2 "Resistors_ThroughHole:Resistor_Horizontal_RM10mm" V 5980 5700 50  0001 C CNN
 F 3 "" H 6050 5700 50  0000 C CNN
 	1    6050 5700
@@
 F 0 "R16" V 6130 5900 50  0000 C CNN
 F 1 "10k" V 6050 5900 50  0000 C CNN
-F 2 "" V 5980 5900 50  0000 C CNN
+F 2 "Resistors_ThroughHole:Resistor_Horizontal_RM10mm" V 5980 5900 50  0001 C CNN
 F 3 "" H 6050 5900 50  0000 C CNN
 	1    6050 5900
@@
 F 0 "R10" V 2680 3850 50  0000 C CNN
 F 1 "1k" V 2600 3850 50  0000 C CNN
-F 2 "" V 2530 3850 50  0000 C CNN
+F 2 "Resistors_ThroughHole:Resistor_Horizontal_RM10mm" V 2530 3850 50  0001 C CNN
 F 3 "" H 2600 3850 50  0000 C CNN
 	1    2600 3850
@@
 	2600 4000 2600 4100
 Connection ~ 2600 4100
+Text GLabel 3300 3100 0    60   Output ~ 0
+/HALT
+Wire Wire Line
+	3300 3100 3400 3100
 $EndSCHEMATC

Commit message: Before removing DFROBOT.
Parts:
- added C4, C5: 0.1 µF, symbol C
Connections:
- net +5V: now also C4.1, C5.1
- net GND: now also C4.2, C5.2
Changed lines of the file:
@@
 $EndDescr
 $Comp
-L GND #PWR029
+L GND #PWR32
 U 1 1 568DE0B3
 P 4100 4600
-F 0 "#PWR029" H 4100 4350 50  0001 C CNN
+F 0 "#PWR32" H 4100 4350 50  0001 C CNN
 F 1 "GND" H 4100 4450 50  0000 C CNN
 F 2 "" H 4100 4600 50  0000 C CNN
@@
 $EndComp
 $Comp
-L +5V #PWR030
+L +5V #PWR31
 U 1 1 568DE0CB
-P 4100 1400
-F 0 "#PWR030" H 4100 1250 50  0001 C CNN
-F 1 "+5V" H 4100 1540 50  0000 C CNN
-F 2 "" H 4100 1400 50  0000 C CNN
-F 3 "" H 4100 1400 50  0000 C CNN
-	1    4100 1400
+P 4100 800
+F 0 "#PWR31" H 4100 650 50  0001 C CNN
+F 1 "+5V" H 4100 940 50  0000 C CNN
+F 2 "" H 4100 800 50  0000 C CNN
+F 3 "" H 4100 800 50  0000 C CNN
+	1    4100 800
 	1    0    0    -1
 $EndComp
@@
 	4100 4600 4100 4500
 Wire Wire Line
-	4100 1500 4100 1400
+	4100 1500 4100 800
 Wire Wire Line
 	4800 3500 4900 3500
@@
 D0
 $Comp
-L +5V #PWR031
+L +5V #PWR30
 U 1 1 568DE771
 P 3200 2350
-F 0 "#PWR031" H 3200 2200 50  0001 C CNN
+F 0 "#PWR30" H 3200 2200 50  0001 C CNN
 F 1 "+5V" H 3200 2490 50  0000 C CNN
 F 2 "" H 3200 2350 50  0000 C CNN
@@
 /Z80_RESET
 $Comp
-L GND #PWR032
+L GND #PWR28
 U 1 1 568DF463
 P 2200 2600
-F 0 "#PWR032" H 2200 2350 50  0001 C CNN
+F 0 "#PWR28" H 2200 2350 50  0001 C CNN
 F 1 "GND" H 2200 2450 50  0000 C CNN
 F 2 "" H 2200 2600 50  0000 C CNN
@@
 A0
 $Comp
-L +5V #PWR033
+L +5V #PWR35
 U 1 1 568E215B
 P 5950 4100
-F 0 "#PWR033" H 5950 3950 50  0001 C CNN
+F 0 "#PWR35" H 5950 3950 50  0001 C CNN
 F 1 "+5V" H 5950 4240 50  0000 C CNN
 F 2 "" H 5950 4100 60  0000 C CNN
@@
 D0
 $Comp
-L +5V #PWR034
+L +5V #PWR39
 U 1 1 568E25EC
-P 8200 3150
-F 0 "#PWR034" H 8200 3000 50  0001 C CNN
-F 1 "+5V" H 8200 3290 50  0000 C CNN
-F 2 "" H 8200 3150 60  0000 C CNN
-F 3 "" H 8200 3150 60  0000 C CNN
-	1    8200 3150
-	1    0    0    -1
-$EndComp
-Wire Wire Line
-	8200 3150 8150 3150
-$Comp
-L GND #PWR035
+P 8750 3150
+F 0 "#PWR39" H 8750 3000 50  0001 C CNN
+F 1 "+5V" H 8750 3290 50  0000 C CNN
+F 2 "" H 8750 3150 60  0000 C CNN
+F 3 "" H 8750 3150 60  0000 C CNN
+	1    8750 3150
+	1    0    0    -1
+$EndComp
+Wire Wire Line
+	8750 3150 8150 3150
+$Comp
+L GND #PWR37
 U 1 1 568E2687
 P 8200 3250
-F 0 "#PWR035" H 8200 3000 50  0001 C CNN
+F 0 "#PWR37" H 8200 3000 50  0001 C CNN
 F 1 "GND" H 8200 3100 50  0000 C CNN
 F 2 "" H 8200 3250 60  0000 C CNN
@@
 	8150 3250 8200 3250
 $Comp
-L GND #PWR036
+L GND #PWR34
 U 1 1 568E2BE1
 P 5750 3800
-F 0 "#PWR036" H 5750 3550 50  0001 C CNN
+F 0 "#PWR34" H 5750 3550 50  0001 C CNN
 F 1 "GND" H 5750 3650 50  0000 C CNN
 F 2 "" H 5750 3800 60  0000 C CNN
@@
 $EndComp
 $Comp
-L GND #PWR037
+L GND #PWR36
 U 1 1 56A01480
 P 6350 5950
-F 0 "#PWR037" H 6350 5700 50  0001 C CNN
+F 0 "#PWR36" H 6350 5700 50  0001 C CNN
 F 1 "GND" H 6350 5800 50  0000 C CNN
 F 2 "" H 6350 5950 50  0000 C CNN
@@
 $EndComp
 Wire Wire Line
-	6350 5950 6350 4900
+	6350 4900 6350 5950
 Wire Wire Line
 	6350 4900 6200 4900
@@
 $EndComp
 $Comp
-L +5V #PWR038
+L +5V #PWR29
 U 1 1 56A02BCE
 P 2600 3600
-F 0 "#PWR038" H 2600 3450 50  0001 C CNN
+F 0 "#PWR29" H 2600 3450 50  0001 C CNN
 F 1 "+5V" H 2600 3740 50  0000 C CNN
 F 2 "" H 2600 3600 60  0000 C CNN
@@
 Wire Wire Line
 	3300 3100 3400 3100
+$Comp
+L GND #PWR33
+U 1 1 56A06CAB
+P 4450 1200
+F 0 "#PWR33" H 4450 950 50  0001 C CNN
+F 1 "GND" H 4450 1050 50  0000 C CNN
+F 2 "" H 4450 1200 50  0000 C CNN
+F 3 "" H 4450 1200 50  0000 C CNN
+	1    4450 1200
+	1    0    0    -1
+$EndComp
+$Comp
+L C C4
+U 1 1 56A06CFE
+P 4450 1000
+F 0 "C4" H 4475 1100 50  0000 L CNN
+F 1 "0.1 µF" H 4475 900 50  0000 L CNN
+F 2 "" H 4488 850 50  0000 C CNN
+F 3 "" H 4450 1000 50  0000 C CNN
+	1    4450 1000
+	1    0    0    -1
+$EndComp
+Wire Wire Line
+	4450 1200 4450 1150
+Wire Wire Line
+	4100 800  4450 800
+Wire Wire Line
+	4450 800  4450 850
+$Comp
+L C C5
+U 1 1 56A06F35
+P 8600 3450
+F 0 "C5" H 8625 3550 50  0000 L CNN
+F 1 "0.1 µF" H 8625 3350 50  0000 L CNN
+F 2 "" H 8638 3300 50  0000 C CNN
+F 3 "" H 8600 3450 50  0000 C CNN
+	1    8600 3450
+	1    0    0    -1
+$EndComp
+$Comp
+L GND #PWR38
+U 1 1 56A06F73
+P 8600 3700
+F 0 "#PWR38" H 8600 3450 50  0001 C CNN
+F 1 "GND" H 8600 3550 50  0000 C CNN
+F 2 "" H 8600 3700 50  0000 C CNN
+F 3 "" H 8600 3700 50  0000 C CNN
+	1    8600 3700
+	1    0    0    -1
+$EndComp
+Wire Wire Line
+	8600 3700 8600 3600
+Wire Wire Line
+	8600 3300 8600 3150
+Connection ~ 8600 3150
 $EndSCHEMATC

Commit message: Remove DFROBOT and LDO.
Parts:
- C4, C5: footprint (none) -> Capacitors_ThroughHole:C_Disc_D6_P5
Changed lines of the file:
@@
 $EndDescr
 $Comp
-L GND #PWR32
+L GND #PWR029
 U 1 1 568DE0B3
 P 4100 4600
-F 0 "#PWR32" H 4100 4350 50  0001 C CNN
+F 0 "#PWR029" H 4100 4350 50  0001 C CNN
 F 1 "GND" H 4100 4450 50  0000 C CNN
 F 2 "" H 4100 4600 50  0000 C CNN
@@
 $EndComp
 $Comp
-L +5V #PWR31
+L +5V #PWR030
 U 1 1 568DE0CB
 P 4100 800
-F 0 "#PWR31" H 4100 650 50  0001 C CNN
+F 0 "#PWR030" H 4100 650 50  0001 C CNN
 F 1 "+5V" H 4100 940 50  0000 C CNN
 F 2 "" H 4100 800 50  0000 C CNN
@@
 D0
 $Comp
-L +5V #PWR30
+L +5V #PWR031
 U 1 1 568DE771
 P 3200 2350
-F 0 "#PWR30" H 3200 2200 50  0001 C CNN
+F 0 "#PWR031" H 3200 2200 50  0001 C CNN
 F 1 "+5V" H 3200 2490 50  0000 C CNN
 F 2 "" H 3200 2350 50  0000 C CNN
@@
 /Z80_RESET
 $Comp
-L GND #PWR28
+L GND #PWR032
 U 1 1 568DF463
 P 2200 2600
-F 0 "#PWR28" H 2200 2350 50  0001 C CNN
+F 0 "#PWR032" H 2200 2350 50  0001 C CNN
 F 1 "GND" H 2200 2450 50  0000 C CNN
 F 2 "" H 2200 2600 50  0000 C CNN
@@
 A0
 $Comp
-L +5V #PWR35
+L +5V #PWR033
 U 1 1 568E215B
 P 5950 4100
-F 0 "#PWR35" H 5950 3950 50  0001 C CNN
+F 0 "#PWR033" H 5950 3950 50  0001 C CNN
 F 1 "+5V" H 5950 4240 50  0000 C CNN
 F 2 "" H 5950 4100 60  0000 C CNN
@@
 D0
 $Comp
-L +5V #PWR39
+L +5V #PWR034
 U 1 1 568E25EC
 P 8750 3150
-F 0 "#PWR39" H 8750 3000 50  0001 C CNN
+F 0 "#PWR034" H 8750 3000 50  0001 C CNN
 F 1 "+5V" H 8750 3290 50  0000 C CNN
 F 2 "" H 8750 3150 60  0000 C CNN
@@
 	8750 3150 8150 3150
 $Comp
-L GND #PWR37
+L GND #PWR035
 U 1 1 568E2687
 P 8200 3250
-F 0 "#PWR37" H 8200 3000 50  0001 C CNN
+F 0 "#PWR035" H 8200 3000 50  0001 C CNN
 F 1 "GND" H 8200 3100 50  0000 C CNN
 F 2 "" H 8200 3250 60  0000 C CNN
@@
 	8150 3250 8200 3250
 $Comp
-L GND #PWR34
+L GND #PWR036
 U 1 1 568E2BE1
 P 5750 3800
-F 0 "#PWR34" H 5750 3550 50  0001 C CNN
+F 0 "#PWR036" H 5750 3550 50  0001 C CNN
 F 1 "GND" H 5750 3650 50  0000 C CNN
 F 2 "" H 5750 3800 60  0000 C CNN
@@
 $EndComp
 $Comp
-L GND #PWR36
+L GND #PWR037
 U 1 1 56A01480
 P 6350 5950
-F 0 "#PWR36" H 6350 5700 50  0001 C CNN
+F 0 "#PWR037" H 6350 5700 50  0001 C CNN
 F 1 "GND" H 6350 5800 50  0000 C CNN
 F 2 "" H 6350 5950 50  0000 C CNN
@@
 $EndComp
 $Comp
-L +5V #PWR29
+L +5V #PWR038
 U 1 1 56A02BCE
 P 2600 3600
-F 0 "#PWR29" H 2600 3450 50  0001 C CNN
+F 0 "#PWR038" H 2600 3450 50  0001 C CNN
 F 1 "+5V" H 2600 3740 50  0000 C CNN
 F 2 "" H 2600 3600 60  0000 C CNN
@@
 	3300 3100 3400 3100
 $Comp
-L GND #PWR33
+L GND #PWR039
 U 1 1 56A06CAB
 P 4450 1200
-F 0 "#PWR33" H 4450 950 50  0001 C CNN
+F 0 "#PWR039" H 4450 950 50  0001 C CNN
 F 1 "GND" H 4450 1050 50  0000 C CNN
 F 2 "" H 4450 1200 50  0000 C CNN
@@
 F 0 "C4" H 4475 1100 50  0000 L CNN
 F 1 "0.1 µF" H 4475 900 50  0000 L CNN
-F 2 "" H 4488 850 50  0000 C CNN
+F 2 "Capacitors_ThroughHole:C_Disc_D6_P5" H 4488 850 50  0001 C CNN
 F 3 "" H 4450 1000 50  0000 C CNN
 	1    4450 1000
@@
 F 0 "C5" H 8625 3550 50  0000 L CNN
 F 1 "0.1 µF" H 8625 3350 50  0000 L CNN
-F 2 "" H 8638 3300 50  0000 C CNN
+F 2 "Capacitors_ThroughHole:C_Disc_D6_P5" H 8638 3300 50  0001 C CNN
 F 3 "" H 8600 3450 50  0000 C CNN
 	1    8600 3450
@@
 $EndComp
 $Comp
-L GND #PWR38
+L GND #PWR040
 U 1 1 56A06F73
 P 8600 3700
-F 0 "#PWR38" H 8600 3450 50  0001 C CNN
+F 0 "#PWR040" H 8600 3450 50  0001 C CNN
 F 1 "GND" H 8600 3550 50  0000 C CNN
 F 2 "" H 8600 3700 50  0000 C CNN
