File: alice3/kicad/MOBO/CPU.sch (KiCad schematic (older format))
At the start: 12 parts, among them U8 Z80CPU, U9 KM681000BLP-7

Commit message: Alice 3 v1 schematic and PCB, sent to OSHPark
Connections:
- net +5V renamed +3V3
Changed lines of the file:
@@
-	1    0    0    -1
-$EndComp
-$Comp
-L +5V #PWR030
-U 1 1 568DE0CB
-P 4100 800
-F 0 "#PWR030" H 4100 650 50  0001 C CNN
-F 1 "+5V" H 4100 940 50  0000 C CNN
-F 2 "" H 4100 800 50  0000 C CNN
-F 3 "" H 4100 800 50  0000 C CNN
-	1    4100 800
 	1    0    0    -1
 $EndComp
@@
 Text GLabel 4900 3500 2    60   BiDi ~ 0
 D0
-$Comp
-L +5V #PWR031
-U 1 1 568DE771
-P 3200 2350
-F 0 "#PWR031" H 3200 2200 50  0001 C CNN
-F 1 "+5V" H 3200 2490 50  0000 C CNN
-F 2 "" H 3200 2350 50  0000 C CNN
-F 3 "" H 3200 2350 50  0000 C CNN
-	1    3200 2350
-	1    0    0    -1
-$EndComp
 Wire Wire Line
 	3200 2350 3200 3000
@@
 /Z80_RESET
 $Comp
-L GND #PWR032
+L GND #PWR030
 U 1 1 568DF463
 P 2200 2600
-F 0 "#PWR032" H 2200 2350 50  0001 C CNN
+F 0 "#PWR030" H 2200 2350 50  0001 C CNN
 F 1 "GND" H 2200 2450 50  0000 C CNN
 F 2 "" H 2200 2600 50  0000 C CNN
@@
 U 1 1 568E02F3
 P 7450 3250
+AR Path="/568E02F3" Ref="U9"  Part="1"
+AR Path="/568DDBCB/568E02F3" Ref="U9"  Part="1"
 F 0 "U9" H 7450 4450 50  0000 C CNN
 F 1 "KM681000BLP-7" H 7520 2050 50  0000 C CNN
@@
 Text GLabel 6750 2200 0    60   Input ~ 0
 A0
-$Comp
-L +5V #PWR033
-U 1 1 568E215B
-P 5950 4100
-F 0 "#PWR033" H 5950 3950 50  0001 C CNN
-F 1 "+5V" H 5950 4240 50  0000 C CNN
-F 2 "" H 5950 4100 60  0000 C CNN
-F 3 "" H 5950 4100 60  0000 C CNN
-	1    5950 4100
-	1    0    0    -1
-$EndComp
 Wire Wire Line
 	5950 4100 6750 4100
@@
 D0
 $Comp
-L +5V #PWR034
-U 1 1 568E25EC
-P 8750 3150
-F 0 "#PWR034" H 8750 3000 50  0001 C CNN
-F 1 "+5V" H 8750 3290 50  0000 C CNN
-F 2 "" H 8750 3150 60  0000 C CNN
-F 3 "" H 8750 3150 60  0000 C CNN
-	1    8750 3150
-	1    0    0    -1
-$EndComp
-Wire Wire Line
-	8750 3150 8150 3150
-$Comp
-L GND #PWR035
+L GND #PWR031
 U 1 1 568E2687
 P 8200 3250
-F 0 "#PWR035" H 8200 3000 50  0001 C CNN
+F 0 "#PWR031" H 8200 3000 50  0001 C CNN
 F 1 "GND" H 8200 3100 50  0000 C CNN
 F 2 "" H 8200 3250 60  0000 C CNN
@@
 	8150 3250 8200 3250
 $Comp
-L GND #PWR036
+L GND #PWR032
 U 1 1 568E2BE1
 P 5750 3800
-F 0 "#PWR036" H 5750 3550 50  0001 C CNN
+F 0 "#PWR032" H 5750 3550 50  0001 C CNN
 F 1 "GND" H 5750 3650 50  0000 C CNN
 F 2 "" H 5750 3800 60  0000 C CNN
@@
 $EndComp
 $Comp
-L GND #PWR037
+L GND #PWR033
 U 1 1 56A01480
 P 6350 5950
-F 0 "#PWR037" H 6350 5700 50  0001 C CNN
+F 0 "#PWR033" H 6350 5700 50  0001 C CNN
 F 1 "GND" H 6350 5800 50  0000 C CNN
 F 2 "" H 6350 5950 50  0000 C CNN
@@
 	1    0    0    -1
 $EndComp
-$Comp
-L +5V #PWR038
-U 1 1 56A02BCE
-P 2600 3600
-F 0 "#PWR038" H 2600 3450 50  0001 C CNN
-F 1 "+5V" H 2600 3740 50  0000 C CNN
-F 2 "" H 2600 3600 60  0000 C CNN
-F 3 "" H 2600 3600 60  0000 C CNN
-	1    2600 3600
-	1    0    0    -1
-$EndComp
 Wire Wire Line
 	2600 3600 2600 3700
@@
 	3300 3100 3400 3100
 $Comp
-L GND #PWR039
+L GND #PWR034
 U 1 1 56A06CAB
 P 4450 1200
-F 0 "#PWR039" H 4450 950 50  0001 C CNN
+F 0 "#PWR034" H 4450 950 50  0001 C CNN
 F 1 "GND" H 4450 1050 50  0000 C CNN
 F 2 "" H 4450 1200 50  0000 C CNN
@@
 $EndComp
 $Comp
-L GND #PWR040
+L GND #PWR035
 U 1 1 56A06F73
 P 8600 3700
-F 0 "#PWR040" H 8600 3450 50  0001 C CNN
+F 0 "#PWR035" H 8600 3450 50  0001 C CNN
 F 1 "GND" H 8600 3550 50  0000 C CNN
 F 2 "" H 8600 3700 50  0000 C CNN
@@
 Wire Wire Line
 	8600 3300 8600 3150
+$Comp
+L +3V3 #PWR036
+U 1 1 56A5493F
+P 4100 800
+F 0 "#PWR036" H 4100 650 50  0001 C CNN
+F 1 "+3V3" H 4100 940 50  0000 C CNN
+F 2 "" H 4100 800 60  0000 C CNN
+F 3 "" H 4100 800 60  0000 C CNN
+	1    4100 800
+	1    0    0    -1
+$EndComp
+$Comp
+L +3V3 #PWR037
+U 1 1 56A549BD
+P 8750 3150
+F 0 "#PWR037" H 8750 3000 50  0001 C CNN
+F 1 "+3V3" H 8750 3290 50  0000 C CNN
+F 2 "" H 8750 3150 60  0000 C CNN
+F 3 "" H 8750 3150 60  0000 C CNN
+	1    8750 3150
+	1    0    0    -1
+$EndComp
+$Comp
+L +3V3 #PWR038
+U 1 1 56A55124
+P 5950 4100
+F 0 "#PWR038" H 5950 3950 50  0001 C CNN
+F 1 "+3V3" H 5950 4240 50  0000 C CNN
+F 2 "" H 5950 4100 60  0000 C CNN
+F 3 "" H 5950 4100 60  0000 C CNN
+	1    5950 4100
+	1    0    0    -1
+$EndComp
+$Comp
+L +3V3 #PWR039
+U 1 1 56A55184
+P 3200 2400
+F 0 "#PWR039" H 3200 2250 50  0001 C CNN
+F 1 "+3V3" H 3200 2540 50  0000 C CNN
+F 2 "" H 3200 2400 60  0000 C CNN
+F 3 "" H 3200 2400 60  0000 C CNN
+	1    3200 2400
+	1    0    0    -1
+$EndComp
+$Comp
+L +3V3 #PWR040
+U 1 1 56A551C0
+P 2600 3600
+F 0 "#PWR040" H 2600 3450 50  0001 C CNN
+F 1 "+3V3" H 2600 3740 50  0000 C CNN
+F 2 "" H 2600 3600 60  0000 C CNN
+F 3 "" H 2600 3600 60  0000 C CNN
+	1    2600 3600
+	1    0    0    -1
+$EndComp
 Connection ~ 8600 3150
+$Comp
+L +3V3 #PWR041
+U 1 1 56A56C3B
+P 8450 3150
+F 0 "#PWR041" H 8450 3000 50  0001 C CNN
+F 1 "+3V3" H 8450 3290 50  0000 C CNN
+F 2 "" H 8450 3150 60  0000 C CNN
+F 3 "" H 8450 3150 60  0000 C CNN
+	1    8450 3150
+	1    0    0    -1
+$EndComp
+Wire Wire Line
+	8600 3150 8750 3150
+Wire Wire Line
+	8150 3150 8450 3150
 $EndSCHEMATC
