File: alice3/kicad/MOBO/IO.sch (KiCad schematic (older format))
At the start: 19 parts, among them CON1 SD_Card, U10 LEVELCONVERTER, U11 LEVELCONVERTER, U6 MiniM4-D40, U7 DFROBOT_FTDI_BASIC, U8 LEVELCONVERTER, U9 LEVELCONVERTER

Commit message: first draft completed integration
Parts:
- gave numbers to parts that had none: 1
- renumbered C2 to C3, D1 to D3, D2 to D4, D3 to D5
Connections:
- wire segments 121 -> 119
- no-connect marks 28 -> 34
Changed lines of the file:
@@
 LIBS:vga_daughter_board
 LIBS:Zilog
+LIBS:km681000blp-7
+LIBS:28f512
 LIBS:MOBO-cache
 EELAYER 25 0
@@
 $EndComp
 $Comp
-L +3.3V #PWR020
+L +3.3V #PWR018
 U 1 1 5689970E
 P 2400 1700
-F 0 "#PWR020" H 2400 1550 50  0001 C CNN
+F 0 "#PWR018" H 2400 1550 50  0001 C CNN
 F 1 "+3.3V" H 2400 1840 50  0000 C CNN
 F 2 "" H 2400 1700 60  0000 C CNN
@@
 $EndComp
 $Comp
-L GND #PWR021
+L GND #PWR019
 U 1 1 5689975D
 P 2400 4600
-F 0 "#PWR021" H 2400 4350 50  0001 C CNN
+F 0 "#PWR019" H 2400 4350 50  0001 C CNN
 F 1 "GND" H 2400 4450 50  0000 C CNN
 F 2 "" H 2400 4600 60  0000 C CNN
@@
 NoConn ~ 2900 6500
 $Comp
-L GND #PWR022
+L GND #PWR020
 U 1 1 56899C9B
 P 3800 7700
-F 0 "#PWR022" H 3800 7450 50  0001 C CNN
+F 0 "#PWR020" H 3800 7450 50  0001 C CNN
 F 1 "GND" H 3800 7550 50  0000 C CNN
 F 2 "" H 3800 7700 60  0000 C CNN
@@
 $EndComp
 $Comp
-L +3.3V #PWR023
+L +3.3V #PWR021
 U 1 1 56899CD4
 P 3900 5850
-F 0 "#PWR023" H 3900 5700 50  0001 C CNN
+F 0 "#PWR021" H 3900 5700 50  0001 C CNN
 F 1 "+3.3V" H 3900 5990 50  0000 C CNN
 F 2 "" H 3900 5850 60  0000 C CNN
@@
 F 3 "" H 3650 6300 30  0000 C CNN
 	1    3650 6300
-	1    0    0    -1
-$EndComp
-$Comp
-L PWR_FLAG #FLG024
-U 1 1 5689EBB4
-P 850 1050
-F 0 "#FLG024" H 850 1145 50  0001 C CNN
-F 1 "PWR_FLAG" H 850 1230 50  0000 C CNN
-F 2 "" H 850 1050 60  0000 C CNN
-F 3 "" H 850 1050 60  0000 C CNN
-	1    850  1050
-	1    0    0    -1
-$EndComp
-$Comp
-L PWR_FLAG #FLG025
-U 1 1 5689EC00
-P 1400 1050
-F 0 "#FLG025" H 1400 1145 50  0001 C CNN
-F 1 "PWR_FLAG" H 1400 1230 50  0000 C CNN
-F 2 "" H 1400 1050 60  0000 C CNN
-F 3 "" H 1400 1050 60  0000 C CNN
-	1    1400 1050
-	1    0    0    -1
-$EndComp
-$Comp
-L +5V #PWR026
-U 1 1 5689EC5C
-P 850 1200
-F 0 "#PWR026" H 850 1050 50  0001 C CNN
-F 1 "+5V" H 850 1340 50  0000 C CNN
-F 2 "" H 850 1200 60  0000 C CNN
-F 3 "" H 850 1200 60  0000 C CNN
-	1    850  1200
-	-1   0    0    1
-$EndComp
-$Comp
-L GND #PWR027
-U 1 1 5689EC88
-P 1400 1200
-F 0 "#PWR027" H 1400 950 50  0001 C CNN
-F 1 "GND" H 1400 1050 50  0000 C CNN
-F 2 "" H 1400 1200 60  0000 C CNN
-F 3 "" H 1400 1200 60  0000 C CNN
-	1    1400 1200
 	1    0    0    -1
 $EndComp
@@
 DI
 $Comp
-L GND #PWR028
+L GND #PWR022
 U 1 1 568A381B
 P 8400 1350
-F 0 "#PWR028" H 8400 1100 50  0001 C CNN
+F 0 "#PWR022" H 8400 1100 50  0001 C CNN
 F 1 "GND" H 8400 1200 50  0000 C CNN
 F 2 "" H 8400 1350 60  0000 C CNN
@@
 $EndComp
 $Comp
-L GND #PWR029
+L GND #PWR023
 U 1 1 568A3851
 P 8400 2400
-F 0 "#PWR029" H 8400 2150 50  0001 C CNN
+F 0 "#PWR023" H 8400 2150 50  0001 C CNN
 F 1 "GND" H 8400 2250 50  0000 C CNN
 F 2 "" H 8400 2400 60  0000 C CNN
@@
 $EndComp
 $Comp
-L GND #PWR030
+L GND #PWR024
 U 1 1 568A3880
 P 8400 3450
-F 0 "#PWR030" H 8400 3200 50  0001 C CNN
+F 0 "#PWR024" H 8400 3200 50  0001 C CNN
 F 1 "GND" H 8400 3300 50  0000 C CNN
 F 2 "" H 8400 3450 60  0000 C CNN
@@
 $EndComp
 $Comp
-L GND #PWR031
+L GND #PWR025
 U 1 1 568A38AF
 P 8400 4500
-F 0 "#PWR031" H 8400 4250 50  0001 C CNN
+F 0 "#PWR025" H 8400 4250 50  0001 C CNN
 F 1 "GND" H 8400 4350 50  0000 C CNN
 F 2 "" H 8400 4500 60  0000 C CNN
@@
 $EndComp
 $Comp
-L GND #PWR032
+L GND #PWR026
 U 1 1 568A38E0
 P 9300 1350
-F 0 "#PWR032" H 9300 1100 50  0001 C CNN
+F 0 "#PWR026" H 9300 1100 50  0001 C CNN
 F 1 "GND" H 9300 1200 50  0000 C CNN
 F 2 "" H 9300 1350 60  0000 C CNN
@@
 $EndComp
 $Comp
-L GND #PWR033
+L GND #PWR027
 U 1 1 568A3916
 P 9300 2400
-F 0 "#PWR033" H 9300 2150 50  0001 C CNN
+F 0 "#PWR027" H 9300 2150 50  0001 C CNN
 F 1 "GND" H 9300 2250 50  0000 C CNN
 F 2 "" H 9300 2400 60  0000 C CNN
@@
 $EndComp
 $Comp
-L GND #PWR034
+L GND #PWR028
 U 1 1 568A3945
 P 9300 3450
-F 0 "#PWR034" H 9300 3200 50  0001 C CNN
+F 0 "#PWR028" H 9300 3200 50  0001 C CNN
 F 1 "GND" H 9300 3300 50  0000 C CNN
 F 2 "" H 9300 3450 60  0000 C CNN
@@
 $EndComp
 $Comp
-L GND #PWR035
+L GND #PWR029
 U 1 1 568A3974
 P 9300 4500
-F 0 "#PWR035" H 9300 4250 50  0001 C CNN
+F 0 "#PWR029" H 9300 4250 50  0001 C CNN
 F 1 "GND" H 9300 4350 50  0000 C CNN
 F 2 "" H 9300 4500 60  0000 C CNN
@@
 $EndComp
 $Comp
-L +3.3V #PWR036
+L +3.3V #PWR030
 U 1 1 568A39A5
 P 8300 1250
-F 0 "#PWR036" H 8300 1100 50  0001 C CNN
+F 0 "#PWR030" H 8300 1100 50  0001 C CNN
 F 1 "+3.3V" H 8300 1390 50  0000 C CNN
 F 2 "" H 8300 1250 60  0000 C CNN
@@
 $EndComp
 $Comp
-L +3.3V #PWR037
+L +3.3V #PWR031
 U 1 1 568A39DB
 P 8300 2300
-F 0 "#PWR037" H 8300 2150 50  0001 C CNN
+F 0 "#PWR031" H 8300 2150 50  0001 C CNN
 F 1 "+3.3V" H 8300 2440 50  0000 C CNN
 F 2 "" H 8300 2300 60  0000 C CNN
@@
 $EndComp
 $Comp
-L +3.3V #PWR038
+L +3.3V #PWR032
 U 1 1 568A3A0A
 P 8300 3350
-F 0 "#PWR038" H 8300 3200 50  0001 C CNN
+F 0 "#PWR032" H 8300 3200 50  0001 C CNN
 F 1 "+3.3V" H 8300 3490 50  0000 C CNN
 F 2 "" H 8300 3350 60  0000 C CNN
@@
 $EndComp
 $Comp
-L +3.3V #PWR039
+L +3.3V #PWR033
 U 1 1 568A3A45
 P 8300 4400
-F 0 "#PWR039" H 8300 4250 50  0001 C CNN
+F 0 "#PWR033" H 8300 4250 50  0001 C CNN
 F 1 "+3.3V" H 8300 4540 50  0000 C CNN
 F 2 "" H 8300 4400 60  0000 C CNN
@@
 $EndComp
 $Comp
-L +5V #PWR040
+L +5V #PWR034
 U 1 1 568A3D49
 P 9400 4400
-F 0 "#PWR040" H 9400 4250 50  0001 C CNN
+F 0 "#PWR034" H 9400 4250 50  0001 C CNN
 F 1 "+5V" H 9400 4540 50  0000 C CNN
 F 2 "" H 9400 4400 60  0000 C CNN
@@
 $EndComp
 $Comp
-L +5V #PWR041
+L +5V #PWR035
 U 1 1 568A3D7F
 P 9400 3350
-F 0 "#PWR041" H 9400 3200 50  0001 C CNN
+F 0 "#PWR035" H 9400 3200 50  0001 C CNN
 F 1 "+5V" H 9400 3490 50  0000 C CNN
 F 2 "" H 9400 3350 60  0000 C CNN
@@
 $EndComp
 $Comp
-L +5V #PWR042
+L +5V #PWR036
 U 1 1 568A3DAE
 P 9400 2300
-F 0 "#PWR042" H 9400 2150 50  0001 C CNN
+F 0 "#PWR036" H 9400 2150 50  0001 C CNN
 F 1 "+5V" H 9400 2440 50  0000 C CNN
 F 2 "" H 9400 2300 60  0000 C CNN
@@
 $EndComp
 $Comp
-L +5V #PWR043
+L +5V #PWR037
 U 1 1 568A3DF5
 P 9400 1250
-F 0 "#PWR043" H 9400 1100 50  0001 C CNN
+F 0 "#PWR037" H 9400 1100 50  0001 C CNN
 F 1 "+5V" H 9400 1390 50  0000 C CNN
 F 2 "" H 9400 1250 60  0000 C CNN
@@
 $EndComp
 $Comp
-L LED D3
+L LED D5
 U 1 1 568A06A4
 P 5100 3350
-F 0 "D3" H 5100 3450 50  0000 C CNN
+F 0 "D5" H 5100 3450 50  0000 C CNN
 F 1 "HEART" H 5250 3300 50  0000 C CNN
 F 2 "LEDs:LED-5MM" H 5250 3300 50  0001 C CNN
@@
 $EndComp
 $Comp
-L LED D2
+L LED D4
 U 1 1 568A071D
 P 1250 4000
-F 0 "D2" H 1250 4100 50  0000 C CNN
+F 0 "D4" H 1250 4100 50  0000 C CNN
 F 1 "PANIC" H 1400 3950 50  0000 C CNN
 F 2 "LEDs:LED-5MM" H 1400 3950 50  0001 C CNN
@@
 $EndComp
 $Comp
-L LED D1
+L LED D3
 U 1 1 568A0E8E
 P 950 4000
-F 0 "D1" H 950 4100 50  0000 C CNN
+F 0 "D3" H 950 4100 50  0000 C CNN
 F 1 "INFO" H 1100 3950 50  0000 C CNN
 F 2 "LEDs:LED-5MM" H 950 4000 50  0001 C CNN
@@
 $EndComp
 $Comp
-L GND #PWR044
+L GND #PWR038
 U 1 1 568A10FA
 P 950 4500
-F 0 "#PWR044" H 950 4250 50  0001 C CNN
+F 0 "#PWR038" H 950 4250 50  0001 C CNN
 F 1 "GND" H 950 4350 50  0000 C CNN
 F 2 "" H 950 4500 60  0000 C CNN
@@
 $EndComp
 $Comp
-L GND #PWR045
+L GND #PWR039
 U 1 1 568A1142
 P 1250 4500
-F 0 "#PWR045" H 1250 4250 50  0001 C CNN
+F 0 "#PWR039" H 1250 4250 50  0001 C CNN
 F 1 "GND" H 1250 4350 50  0000 C CNN
 F 2 "" H 1250 4500 60  0000 C CNN
@@
 $EndComp
 $Comp
-L GND #PWR046
+L GND #PWR040
 U 1 1 568A1183
 P 5100 3850
-F 0 "#PWR046" H 5100 3600 50  0001 C CNN
+F 0 "#PWR040" H 5100 3600 50  0001 C CNN
 F 1 "GND" H 5100 3700 50  0000 C CNN
 F 2 "" H 5100 3850 60  0000 C CNN
@@
 $EndComp
 $Comp
-L GND #PWR047
+L GND #PWR041
 U 1 1 568A2172
 P 5650 2550
-F 0 "#PWR047" H 5650 2300 50  0001 C CNN
+F 0 "#PWR041" H 5650 2300 50  0001 C CNN
 F 1 "GND" H 5650 2400 50  0000 C CNN
 F 2 "" H 5650 2550 60  0000 C CNN
@@
 $EndComp
 $Comp
-L GND #PWR048
+L GND #PWR042
 U 1 1 568A21B9
 P 6650 3150
-F 0 "#PWR048" H 6650 2900 50  0001 C CNN
+F 0 "#PWR042" H 6650 2900 50  0001 C CNN
 F 1 "GND" H 6650 3000 50  0000 C CNN
 F 2 "" H 6650 3150 60  0000 C CNN
@@
 NoConn ~ 4000 2200
 $Comp
-L CP1 C2
+L CP1 C3
 U 1 1 568A9C8C
 P 3600 7600
-F 0 "C2" H 3625 7700 50  0000 L CNN
+F 0 "C3" H 3625 7700 50  0000 L CNN
 F 1 "22µF" H 3625 7500 50  0000 L CNN
 F 2 "Capacitors_ThroughHole:C_Radial_D5_L11_P2" H 3600 7600 60  0001 C CNN
@@
 $EndComp
 $Comp
-L +5V #PWR049
+L +5V #PWR043
 U 1 1 568DC45F
 P 7000 2650
-F 0 "#PWR049" H 7000 2500 50  0001 C CNN
+F 0 "#PWR043" H 7000 2500 50  0001 C CNN
 F 1 "+5V" H 7000 2790 50  0000 C CNN
 F 2 "" H 7000 2650 60  0000 C CNN
@@
 /WAIT_5v
 $Comp
-L LEVELCONVERTER U?
+L LEVELCONVERTER U12
 U 1 1 568DD592
 P 8850 5500
-F 0 "U?" H 8700 5950 60  0000 C CNN
+F 0 "U12" H 8700 5950 60  0000 C CNN
 F 1 "LEVELCONVERTER" H 8950 5050 60  0000 C CNN
 F 2 "level converter:LEVELCONV" H 8850 4650 60  0001 C CNN
@@
 /BUSACK_5v
 $Comp
-L +3.3V #PWR?
+L +3.3V #PWR044
 U 1 1 568DDB7F
 P 8300 5450
-F 0 "#PWR?" H 8300 5300 50  0001 C CNN
+F 0 "#PWR044" H 8300 5300 50  0001 C CNN
 F 1 "+3.3V" H 8300 5590 50  0000 C CNN
 F 2 "" H 8300 5450 60  0000 C CNN
@@
 $EndComp
 $Comp
-L GND #PWR?
+L GND #PWR045
 U 1 1 568DDBC3
 P 8400 5550
-F 0 "#PWR?" H 8400 5300 50  0001 C CNN
+F 0 "#PWR045" H 8400 5300 50  0001 C CNN
 F 1 "GND" H 8400 5400 50  0000 C CNN
 F 2 "" H 8400 5550 60  0000 C CNN
@@
 $EndComp
 $Comp
-L GND #PWR?
+L GND #PWR046
 U 1 1 568DDD13
 P 9300 5550
-F 0 "#PWR?" H 9300 5300 50  0001 C CNN
+F 0 "#PWR046" H 9300 5300 50  0001 C CNN
 F 1 "GND" H 9300 5400 50  0000 C CNN
 F 2 "" H 9300 5550 60  0000 C CNN
@@
 $EndComp
 $Comp
-L +5V #PWR?
+L +5V #PWR047
 U 1 1 568DDD57
 P 9400 5450
-F 0 "#PWR?" H 9400 5300 50  0001 C CNN
+F 0 "#PWR047" H 9400 5300 50  0001 C CNN
 F 1 "+5V" H 9400 5590 50  0000 C CNN
 F 2 "" H 9400 5450 60  0000 C CNN
@@
 	3750 7600 3800 7600
 Connection ~ 3800 7600
-Wire Wire Line
-	1400 1050 1400 1200
-Wire Wire Line
-	850  1050 850  1200
 Wire Wire Line
 	2900 7100 4150 7100
@@
 Wire Wire Line
 	9300 5450 9400 5450
+NoConn ~ 8400 5650
+NoConn ~ 8400 5750
+NoConn ~ 9300 5650
+NoConn ~ 9300 5750
+NoConn ~ 9300 4700
+NoConn ~ 8400 4700
 $EndSCHEMATC

Commit message: remove some unused lines, attach +5 to Vcc on 74xx
Parts:
- removed U12: LEVELCONVERTER, level converter:LEVELCONV, symbol LEVELCONVERTER
Connections:
- net labels removed: /M1, /WAIT, /WAIT_5v
- wire segments 119 -> 113
- no-connect marks 34 -> 28
Changed lines of the file:
@@
 $EndDescr
-$Comp
-L MiniM4-D40 U6
-U 1 1 568996B3
-P 3350 3100
-F 0 "U6" H 3000 4550 60  0000 C CNN
-F 1 "MiniM4-D40" H 3350 1650 60  0000 C CNN
-F 2 "Housings_DIP:DIP-40_W15.24mm" H 3200 1600 60  0001 C CNN
-F 3 "" H 3200 1600 60  0000 C CNN
-	1    3350 3100
-	1    0    0    -1
-$EndComp
 $Comp
 L +3.3V #PWR018
@@
 NoConn ~ 4000 3000
 NoConn ~ 4000 2900
-NoConn ~ 4000 2300
-NoConn ~ 4000 2200
 $Comp
 L CP1 C3
@@
 Text GLabel 2450 3100 0    60   BiDi ~ 0
 /WR
-Text GLabel 2450 3500 0    60   Output ~ 0
-/WAIT
 Text GLabel 2450 3900 0    60   BiDi ~ 0
 /RESET
 Text GLabel 2450 4000 0    60   Output ~ 0
 /INT
-Text GLabel 4300 3200 2    60   Input ~ 0
-/M1
 Text GLabel 4300 3300 2    60   BiDi ~ 0
 A7
@@
 Text GLabel 8050 4300 0    60   BiDi ~ 0
 /RESET
-Text GLabel 8050 4600 0    60   Input ~ 0
-/WAIT
 Text GLabel 9750 1050 2    60   BiDi ~ 0
 D0_5v
@@
 Text GLabel 9750 4300 2    60   BiDi ~ 0
 /RESET_5v
-Text GLabel 9750 4600 2    60   Output ~ 0
-/WAIT_5v
-$Comp
-L LEVELCONVERTER U12
-U 1 1 568DD592
-P 8850 5500
-F 0 "U12" H 8700 5950 60  0000 C CNN
-F 1 "LEVELCONVERTER" H 8950 5050 60  0000 C CNN
-F 2 "level converter:LEVELCONV" H 8850 4650 60  0001 C CNN
-F 3 "" H 8850 4650 60  0000 C CNN
-	1    8850 5500
-	1    0    0    -1
-$EndComp
-Text GLabel 8050 5250 0    60   Input ~ 0
+Text GLabel 8050 4600 0    60   Input ~ 0
 /BUSRQ
-Text GLabel 8050 5350 0    60   Output ~ 0
+Text GLabel 8050 4700 0    60   Output ~ 0
 /BUSACK
-Text GLabel 9750 5250 2    60   Output ~ 0
+Text GLabel 9700 4600 2    60   Output ~ 0
 /BUSRQ_5v
-Text GLabel 9750 5350 2    60   Input ~ 0
+Text GLabel 9700 4700 2    60   Input ~ 0
 /BUSACK_5v
-$Comp
-L +3.3V #PWR044
-U 1 1 568DDB7F
-P 8300 5450
-F 0 "#PWR044" H 8300 5300 50  0001 C CNN
-F 1 "+3.3V" H 8300 5590 50  0000 C CNN
-F 2 "" H 8300 5450 60  0000 C CNN
-F 3 "" H 8300 5450 60  0000 C CNN
-	1    8300 5450
-	0    -1   -1   0
-$EndComp
-$Comp
-L GND #PWR045
-U 1 1 568DDBC3
-P 8400 5550
-F 0 "#PWR045" H 8400 5300 50  0001 C CNN
-F 1 "GND" H 8400 5400 50  0000 C CNN
-F 2 "" H 8400 5550 60  0000 C CNN
-F 3 "" H 8400 5550 60  0000 C CNN
-	1    8400 5550
-	0    1    1    0
-$EndComp
-$Comp
-L GND #PWR046
-U 1 1 568DDD13
-P 9300 5550
-F 0 "#PWR046" H 9300 5300 50  0001 C CNN
-F 1 "GND" H 9300 5400 50  0000 C CNN
-F 2 "" H 9300 5550 60  0000 C CNN
-F 3 "" H 9300 5550 60  0000 C CNN
-	1    9300 5550
-	0    -1   -1   0
-$EndComp
-$Comp
-L +5V #PWR047
-U 1 1 568DDD57
-P 9400 5450
-F 0 "#PWR047" H 9400 5300 50  0001 C CNN
-F 1 "+5V" H 9400 5590 50  0000 C CNN
-F 2 "" H 9400 5450 60  0000 C CNN
-F 3 "" H 9400 5450 60  0000 C CNN
-	1    9400 5450
-	0    1    1    0
-$EndComp
 Connection ~ 3800 7000
 Wire Wire Line
@@
 	2700 3100 2450 3100
 Wire Wire Line
-	2450 3500 2700 3500
-Wire Wire Line
 	2700 3900 2450 3900
 Wire Wire Line
@@
 	1650 3300 1850 3300
 Wire Wire Line
-	4000 3200 4300 3200
-Wire Wire Line
 	4000 3300 4300 3300
 Wire Wire Line
@@
 	8050 4300 8400 4300
 Wire Wire Line
+	8400 1250 8300 1250
+Wire Wire Line
+	8400 2300 8300 2300
+Wire Wire Line
+	8400 3350 8300 3350
+Wire Wire Line
+	8300 4400 8400 4400
+Wire Wire Line
+	9400 1250 9300 1250
+Wire Wire Line
+	9300 4400 9400 4400
+Wire Wire Line
+	9400 2300 9300 2300
+Wire Wire Line
+	9400 3350 9300 3350
+Wire Wire Line
+	9300 1050 9750 1050
+Wire Wire Line
+	9750 1150 9300 1150
+Wire Wire Line
+	9300 1450 9750 1450
+Wire Wire Line
+	9750 1550 9300 1550
+Wire Wire Line
+	9300 2100 9750 2100
+Wire Wire Line
+	9750 2200 9300 2200
+Wire Wire Line
+	9300 2500 9750 2500
+Wire Wire Line
+	9750 2600 9300 2600
+Wire Wire Line
+	9750 3150 9300 3150
+Wire Wire Line
+	9300 3250 9750 3250
+Wire Wire Line
+	9750 3550 9300 3550
+Wire Wire Line
+	9300 3650 9750 3650
+Wire Wire Line
+	9300 4200 9750 4200
+Wire Wire Line
+	9750 4300 9300 4300
+Wire Wire Line
+	1850 3800 2700 3800
+Wire Wire Line
+	2700 3700 1250 3700
+Wire Wire Line
+	5100 3100 5100 3150
+Wire Wire Line
+	2700 3600 2550 3600
+Wire Wire Line
+	2550 3600 2550 3650
+Wire Wire Line
+	2550 3650 950  3650
+Wire Wire Line
+	1250 3700 1250 3800
+Wire Wire Line
+	5100 3100 4000 3100
+Wire Wire Line
+	950  3650 950  3800
+Wire Wire Line
+	4200 1400 4200 2800
+Wire Wire Line
+	4200 2800 4000 2800
+Wire Wire Line
+	1750 1200 1750 2950
+Wire Wire Line
+	1750 2950 2450 2950
+Wire Wire Line
+	2450 2950 2450 2900
+Wire Wire Line
+	2450 2900 2700 2900
+Wire Wire Line
+	5650 2750 4600 2750
+Wire Wire Line
+	4600 2750 4600 2600
+Wire Wire Line
+	4600 2600 4000 2600
+Wire Wire Line
+	4000 2700 4500 2700
+Wire Wire Line
+	4500 2700 4500 2900
+Wire Wire Line
+	4500 2900 5500 2900
+Wire Wire Line
+	5500 2900 5500 3150
+Wire Wire Line
+	5500 3150 5650 3150
+Wire Wire Line
+	1750 1200 4400 1200
+Wire Wire Line
+	4200 1400 4400 1400
+Wire Wire Line
+	6650 2850 7000 2850
+Wire Wire Line
+	7000 2850 7000 2650
+Wire Wire Line
+	2400 1700 2400 2000
+Wire Wire Line
+	1850 3300 1850 3800
+Text GLabel 4000 2300 2    60   Output ~ 0
+/BUSRQ
+$Comp
+L MiniM4-D40 U6
+U 1 1 568996B3
+P 3350 3100
+F 0 "U6" H 3000 4550 60  0000 C CNN
+F 1 "MiniM4-D40" H 3350 1650 60  0000 C CNN
+F 2 "Housings_DIP:DIP-40_W15.24mm" H 3200 1600 60  0001 C CNN
+F 3 "" H 3200 1600 60  0000 C CNN
+	1    3350 3100
+	1    0    0    -1
+$EndComp
+Text GLabel 4000 2200 2    60   Input ~ 0
+/BUSACK
+NoConn ~ 4000 3200
+Wire Wire Line
+	9700 4600 9300 4600
+Wire Wire Line
+	9700 4700 9300 4700
+Wire Wire Line
+	8400 4700 8050 4700
+Wire Wire Line
 	8050 4600 8400 4600
-Wire Wire Line
-	8400 1250 8300 1250
-Wire Wire Line
-	8400 2300 8300 2300
-Wire Wire Line
-	8400 3350 8300 3350
-Wire Wire Line
-	8300 4400 8400 4400
-Wire Wire Line
-	9400 1250 9300 1250
-Wire Wire Line
-	9300 4400 9400 4400
-Wire Wire Line
-	9400 2300 9300 2300
-Wire Wire Line
-	9400 3350 9300 3350
-Wire Wire Line
-	9300 1050 9750 1050
-Wire Wire Line
-	9750 1150 9300 1150
-Wire Wire Line
-	9300 1450 9750 1450
-Wire Wire Line
-	9750 1550 9300 1550
-Wire Wire Line
-	9300 2100 9750 2100
-Wire Wire Line
-	9750 2200 9300 2200
-Wire Wire Line
-	9300 2500 9750 2500
-Wire Wire Line
-	9750 2600 9300 2600
-Wire Wire Line
-	9750 3150 9300 3150
-Wire Wire Line
-	9300 3250 9750 3250
-Wire Wire Line
-	9750 3550 9300 3550
-Wire Wire Line
-	9300 3650 9750 3650
-Wire Wire Line
-	9300 4200 9750 4200
-Wire Wire Line
-	9750 4300 9300 4300
-Wire Wire Line
-	9300 4600 9750 4600
-Wire Wire Line
-	1850 3800 2700 3800
-Wire Wire Line
-	2700 3700 1250 3700
-Wire Wire Line
-	5100 3100 5100 3150
-Wire Wire Line
-	2700 3600 2550 3600
-Wire Wire Line
-	2550 3600 2550 3650
-Wire Wire Line
-	2550 3650 950  3650
-Wire Wire Line
-	1250 3700 1250 3800
-Wire Wire Line
-	5100 3100 4000 3100
-Wire Wire Line
-	950  3650 950  3800
-Wire Wire Line
-	4200 1400 4200 2800
-Wire Wire Line
-	4200 2800 4000 2800
-Wire Wire Line
-	1750 1200 1750 2950
-Wire Wire Line
-	1750 2950 2450 2950
-Wire Wire Line
-	2450 2950 2450 2900
-Wire Wire Line
-	2450 2900 2700 2900
-Wire Wire Line
-	5650 2750 4600 2750
-Wire Wire Line
-	4600 2750 4600 2600
-Wire Wire Line
-	4600 2600 4000 2600
-Wire Wire Line
-	4000 2700 4500 2700
-Wire Wire Line
-	4500 2700 4500 2900
-Wire Wire Line
-	4500 2900 5500 2900
-Wire Wire Line
-	5500 2900 5500 3150
-Wire Wire Line
-	5500 3150 5650 3150
-Wire Wire Line
-	1750 1200 4400 1200
-Wire Wire Line
-	4200 1400 4400 1400
-Wire Wire Line
-	6650 2850 7000 2850
-Wire Wire Line
-	7000 2850 7000 2650
-Wire Wire Line
-	2400 1700 2400 2000
-Wire Wire Line
-	1850 3300 1850 3800
-Wire Wire Line
-	9750 5250 9300 5250
-Wire Wire Line
-	9300 5350 9750 5350
-Wire Wire Line
-	8400 5250 8050 5250
-Wire Wire Line
-	8050 5350 8400 5350
-Wire Wire Line
-	8300 5450 8400 5450
-Wire Wire Line
-	9300 5450 9400 5450
-NoConn ~ 8400 5650
-NoConn ~ 8400 5750
-NoConn ~ 9300 5650
-NoConn ~ 9300 5750
-NoConn ~ 9300 4700
-NoConn ~ 8400 4700
+NoConn ~ 2700 3500
 $EndSCHEMATC

Commit message: Sync schematic with breadboard.
Parts:
- removed D3: INFO, LEDs:LED-5MM, symbol LED
- removed D4: PANIC, LEDs:LED-5MM, symbol LED
- removed D5: HEART, LEDs:LED-5MM, symbol LED
- removed R11, R5: 220, Resistors_ThroughHole:Resistor_Horizontal_RM10mm, symbol R
- removed U10, U11, U8, U9: LEVELCONVERTER, level converter:LEVELCONV, symbol LEVELCONVERTER
- added C3: 0.1µ, symbol C
- added SW2: SOFT RESET, symbol SW_PUSH
- added SW3: POWER, symbol SPST
- CON1: footprint Connect:SD_Card_Receptacle -> Sparkfun breakout
- R4: renamed from R6; value 220 -> 10k
- renumbered C3 to C4, R7 to R5, R8 to R6, R9 to R7, R10 to R8
Connections:
- net labels added: /MREQ, /Z80_RESET, A0, A1, A2, A3, A4, A5, A6, A8, A9
- net labels removed: /BUSACK_5v, /BUSRQ_5v, /INT, /INT_5v, /IORQ_5v, /RD_5v, /RESET_5v, /WR_5v, A7_5v, D0_5v, D1_5v, D2_5v, D3_5v, D4_5v, D5_5v, D6_5v, D7_5v
- wire segments 113 -> 75
- no-connect marks 28 -> 18
Other:
- moved on the sheet: C4, R4, R5, R6, R7, R8

Commit message: Start PCB.
Parts:
- C3: footprint (none) -> Capacitors_ThroughHole:C_Disc_D6_P5
- C4: footprint Capacitors_ThroughHole:C_Radial_D5_L11_P2 -> Capacitors_ThroughHole:C_Radial_D5_L11_P2.5
- CON1: footprint Sparkfun breakout -> Pin_Headers:Pin_Header_Straight_1x10
- SW2: footprint (none) -> Buttons_Switches_ThroughHole:SW_PUSH_SMALL
- SW3: footprint (none) -> Buttons_Switches_ThroughHole:SW_SPDT
Connections:
- net labels added: /HALT
- wire segments 75 -> 76
- no-connect marks 18 -> 17
Changed lines of the file:
@@
 F 0 "C4" H 8175 5900 50  0000 L CNN
 F 1 "22µF" H 8175 5700 50  0000 L CNN
-F 2 "Capacitors_ThroughHole:C_Radial_D5_L11_P2" H 8150 5800 60  0001 C CNN
+F 2 "Capacitors_ThroughHole:C_Radial_D5_L11_P2.5" H 8150 5800 60  0001 C CNN
 F 3 "" H 8150 5800 60  0000 C CNN
 	1    8150 5800
@@
 F 0 "SW3" H 7500 2950 50  0000 C CNN
 F 1 "POWER" H 7500 2750 50  0000 C CNN
-F 2 "" H 7500 2850 50  0000 C CNN
+F 2 "Buttons_Switches_ThroughHole:SW_SPDT" H 7500 2850 50  0001 C CNN
 F 3 "" H 7500 2850 50  0000 C CNN
 	1    7500 2850
@@
 F 0 "SW2" H 1050 3410 50  0000 C CNN
 F 1 "SOFT RESET" H 900 3220 50  0000 C CNN
-F 2 "" H 900 3300 50  0000 C CNN
+F 2 "Buttons_Switches_ThroughHole:SW_PUSH_SMALL" H 900 3300 50  0001 C CNN
 F 3 "" H 900 3300 50  0000 C CNN
 	1    900  3300
@@
 F 0 "CON1" H 5900 5600 50  0000 C CNN
 F 1 "SD_Card" H 7150 4500 50  0000 C CNN
-F 2 "Sparkfun breakout" H 6750 5400 50  0000 C CNN
+F 2 "Pin_Headers:Pin_Header_Straight_1x10" H 6750 5400 50  0000 C CNN
 F 3 "" H 6550 5050 50  0000 C CNN
 	1    6550 5050
@@
 Connection ~ 8000 5100
 NoConn ~ 7450 5200
-NoConn ~ 4000 3100
 Text GLabel 4300 3500 2    60   BiDi ~ 0
 A0
@@
 F 0 "C3" H 1775 2050 50  0000 L CNN
 F 1 "0.1µ" H 1775 1850 50  0000 L CNN
-F 2 "" H 1788 1800 50  0000 C CNN
+F 2 "Capacitors_ThroughHole:C_Disc_D6_P5" H 1788 1800 50  0001 C CNN
 F 3 "" H 1750 1950 50  0000 C CNN
 	1    1750 1950
@@
 	1750 1700 2400 1700
 Connection ~ 2400 1700
+Text GLabel 4300 3100 2    60   Input ~ 0
+/HALT
+Wire Wire Line
+	4000 3100 4300 3100
 $EndSCHEMATC
