File: alice3/kicad/MOBO_SMD/CPU.sch (KiCad schematic (older format))
At the start: 12 parts, among them U8 Z80CPU, U9 KM681000BLP-7

Commit message: Run all address lines to ARM UART header
Parts:
- removed R11, R12, R13, R14, R15: 10k, Resistors_ThroughHole:Resistor_Horizontal_RM10mm, symbol R
Connections:
- net labels added: A16
- wire segments 66 -> 55
Other:
- moved on the sheet: R16
Changed lines of the file:
@@
 $EndDescr
 $Comp
-L GND #PWR44
+L GND #PWR042
 U 1 1 568DE0B3
 P 4100 4600
-F 0 "#PWR44" H 4100 4350 50  0001 C CNN
+F 0 "#PWR042" H 4100 4350 50  0001 C CNN
 F 1 "GND" H 4100 4450 50  0000 C CNN
 F 2 "" H 4100 4600 50  0000 C CNN
@@
 /Z80_RESET
 $Comp
-L GND #PWR40
+L GND #PWR043
 U 1 1 568DF463
 P 2200 2600
-F 0 "#PWR40" H 2200 2350 50  0001 C CNN
+F 0 "#PWR043" H 2200 2350 50  0001 C CNN
 F 1 "GND" H 2200 2450 50  0000 C CNN
 F 2 "" H 2200 2600 50  0000 C CNN
@@
 D0
 $Comp
-L GND #PWR49
+L GND #PWR044
 U 1 1 568E2687
 P 8200 3250
-F 0 "#PWR49" H 8200 3000 50  0001 C CNN
+F 0 "#PWR044" H 8200 3000 50  0001 C CNN
 F 1 "GND" H 8200 3100 50  0000 C CNN
 F 2 "" H 8200 3250 60  0000 C CNN
@@
 Wire Wire Line
 	8150 3250 8200 3250
-$Comp
-L GND #PWR46
-U 1 1 568E2BE1
-P 5750 3800
-F 0 "#PWR46" H 5750 3550 50  0001 C CNN
-F 1 "GND" H 5750 3650 50  0000 C CNN
-F 2 "" H 5750 3800 60  0000 C CNN
-F 3 "" H 5750 3800 60  0000 C CNN
-	1    5750 3800
-	1    0    0    -1
-$EndComp
-Wire Wire Line
-	6750 3800 5750 3800
 Text GLabel 3150 2100 0    60   Input ~ 0
 CLK
@@
 Text GLabel 6750 4300 0    60   Input ~ 0
 /WR
-Text GLabel 5800 5900 0    60   Input ~ 0
-A15
-Text GLabel 5800 5700 0    60   Input ~ 0
-A14
-Text GLabel 5800 5500 0    60   Input ~ 0
-A13
-Text GLabel 5800 5300 0    60   Input ~ 0
-A12
-Text GLabel 5800 5100 0    60   Input ~ 0
-A11
-Text GLabel 5800 4900 0    60   Input ~ 0
-A10
-$Comp
-L R R11
-U 1 1 56A0132C
-P 6050 4900
-F 0 "R11" V 6130 4900 50  0000 C CNN
-F 1 "10k" V 6050 4900 50  0000 C CNN
-F 2 "Resistors_ThroughHole:Resistor_Horizontal_RM10mm" V 5980 4900 50  0001 C CNN
-F 3 "" H 6050 4900 50  0000 C CNN
-	1    6050 4900
-	0    1    1    0
-$EndComp
-$Comp
-L R R12
-U 1 1 56A013C6
-P 6050 5100
-F 0 "R12" V 6130 5100 50  0000 C CNN
-F 1 "10k" V 6050 5100 50  0000 C CNN
-F 2 "Resistors_ThroughHole:Resistor_Horizontal_RM10mm" V 5980 5100 50  0001 C CNN
-F 3 "" H 6050 5100 50  0000 C CNN
-	1    6050 5100
-	0    1    1    0
-$EndComp
-$Comp
-L R R13
-U 1 1 56A013E6
-P 6050 5300
-F 0 "R13" V 6130 5300 50  0000 C CNN
-F 1 "10k" V 6050 5300 50  0000 C CNN
-F 2 "Resistors_ThroughHole:Resistor_Horizontal_RM10mm" V 5980 5300 50  0001 C CNN
-F 3 "" H 6050 5300 50  0000 C CNN
-	1    6050 5300
-	0    1    1    0
-$EndComp
-$Comp
-L R R14
-U 1 1 56A01409
-P 6050 5500
-F 0 "R14" V 6130 5500 50  0000 C CNN
-F 1 "10k" V 6050 5500 50  0000 C CNN
-F 2 "Resistors_ThroughHole:Resistor_Horizontal_RM10mm" V 5980 5500 50  0001 C CNN
-F 3 "" H 6050 5500 50  0000 C CNN
-	1    6050 5500
-	0    1    1    0
-$EndComp
-$Comp
-L R R15
-U 1 1 56A0142E
-P 6050 5700
-F 0 "R15" V 6130 5700 50  0000 C CNN
-F 1 "10k" V 6050 5700 50  0000 C CNN
-F 2 "Resistors_ThroughHole:Resistor_Horizontal_RM10mm" V 5980 5700 50  0001 C CNN
-F 3 "" H 6050 5700 50  0000 C CNN
-	1    6050 5700
-	0    1    1    0
-$EndComp
+Text GLabel 5850 4825 0    60   Input ~ 0
+A16
 $Comp
 L R R16
 U 1 1 56A01455
-P 6050 5900
-F 0 "R16" V 6130 5900 50  0000 C CNN
-F 1 "10k" V 6050 5900 50  0000 C CNN
-F 2 "Resistors_ThroughHole:Resistor_Horizontal_RM10mm" V 5980 5900 50  0001 C CNN
-F 3 "" H 6050 5900 50  0000 C CNN
-	1    6050 5900
+P 6100 4825
+F 0 "R16" V 6180 4825 50  0000 C CNN
+F 1 "10k" V 6100 4825 50  0000 C CNN
+F 2 "Resistors_ThroughHole:Resistor_Horizontal_RM10mm" V 6030 4825 50  0001 C CNN
+F 3 "" H 6100 4825 50  0000 C CNN
+	1    6100 4825
 	0    1    1    0
 $EndComp
 $Comp
-L GND #PWR48
+L GND #PWR045
 U 1 1 56A01480
-P 6350 5950
-F 0 "#PWR48" H 6350 5700 50  0001 C CNN
-F 1 "GND" H 6350 5800 50  0000 C CNN
-F 2 "" H 6350 5950 50  0000 C CNN
-F 3 "" H 6350 5950 50  0000 C CNN
-	1    6350 5950
-	1    0    0    -1
-$EndComp
-Wire Wire Line
-	6350 4900 6350 5950
-Wire Wire Line
-	6350 4900 6200 4900
-Wire Wire Line
-	6200 5100 6350 5100
-Connection ~ 6350 5100
-Wire Wire Line
-	6200 5300 6350 5300
-Connection ~ 6350 5300
-Wire Wire Line
-	6200 5500 6350 5500
-Connection ~ 6350 5500
-Wire Wire Line
-	6200 5700 6350 5700
-Connection ~ 6350 5700
-Wire Wire Line
-	6200 5900 6350 5900
-Connection ~ 6350 5900
-Wire Wire Line
-	5800 4900 5900 4900
-Wire Wire Line
-	5800 5100 5900 5100
-Wire Wire Line
-	5800 5300 5900 5300
-Wire Wire Line
-	5800 5500 5900 5500
-Wire Wire Line
-	5800 5700 5900 5700
-Wire Wire Line
-	5800 5900 5900 5900
+P 6400 5050
+F 0 "#PWR045" H 6400 4800 50  0001 C CNN
+F 1 "GND" H 6400 4900 50  0000 C CNN
+F 2 "" H 6400 5050 50  0000 C CNN
+F 3 "" H 6400 5050 50  0000 C CNN
+	1    6400 5050
+	1    0    0    -1
+$EndComp
+Wire Wire Line
+	6250 4825 6400 4825
+Wire Wire Line
+	5850 4825 5950 4825
 $Comp
 L R R10
@@
 	3300 3100 3400 3100
 $Comp
-L GND #PWR45
+L GND #PWR046
 U 1 1 56A06CAB
 P 4450 1200
-F 0 "#PWR45" H 4450 950 50  0001 C CNN
+F 0 "#PWR046" H 4450 950 50  0001 C CNN
 F 1 "GND" H 4450 1050 50  0000 C CNN
 F 2 "" H 4450 1200 50  0000 C CNN
@@
 $EndComp
 $Comp
-L GND #PWR51
+L GND #PWR047
 U 1 1 56A06F73
 P 8600 3700
-F 0 "#PWR51" H 8600 3450 50  0001 C CNN
+F 0 "#PWR047" H 8600 3450 50  0001 C CNN
 F 1 "GND" H 8600 3550 50  0000 C CNN
 F 2 "" H 8600 3700 50  0000 C CNN
@@
 	8600 3300 8600 3150
 $Comp
-L +3V3 #PWR43
+L +3V3 #PWR048
 U 1 1 56A5493F
 P 4100 800
-F 0 "#PWR43" H 4100 650 50  0001 C CNN
+F 0 "#PWR048" H 4100 650 50  0001 C CNN
 F 1 "+3V3" H 4100 940 50  0000 C CNN
 F 2 "" H 4100 800 60  0000 C CNN
@@
 $EndComp
 $Comp
-L +3V3 #PWR52
+L +3V3 #PWR049
 U 1 1 56A549BD
 P 8750 3150
-F 0 "#PWR52" H 8750 3000 50  0001 C CNN
+F 0 "#PWR049" H 8750 3000 50  0001 C CNN
 F 1 "+3V3" H 8750 3290 50  0000 C CNN
 F 2 "" H 8750 3150 60  0000 C CNN
@@
 $EndComp
 $Comp
-L +3V3 #PWR47
+L +3V3 #PWR050
 U 1 1 56A55124
 P 5950 4100
-F 0 "#PWR47" H 5950 3950 50  0001 C CNN
+F 0 "#PWR050" H 5950 3950 50  0001 C CNN
 F 1 "+3V3" H 5950 4240 50  0000 C CNN
 F 2 "" H 5950 4100 60  0000 C CNN
@@
 $EndComp
 $Comp
-L +3V3 #PWR42
+L +3V3 #PWR051
 U 1 1 56A55184
 P 3200 2400
-F 0 "#PWR42" H 3200 2250 50  0001 C CNN
+F 0 "#PWR051" H 3200 2250 50  0001 C CNN
 F 1 "+3V3" H 3200 2540 50  0000 C CNN
 F 2 "" H 3200 2400 60  0000 C CNN
@@
 $EndComp
 $Comp
-L +3V3 #PWR41
+L +3V3 #PWR052
 U 1 1 56A551C0
 P 2600 3600
-F 0 "#PWR41" H 2600 3450 50  0001 C CNN
+F 0 "#PWR052" H 2600 3450 50  0001 C CNN
 F 1 "+3V3" H 2600 3740 50  0000 C CNN
 F 2 "" H 2600 3600 60  0000 C CNN
@@
 Connection ~ 8600 3150
 $Comp
-L +3V3 #PWR50
+L +3V3 #PWR053
 U 1 1 56A56C3B
 P 8450 3150
-F 0 "#PWR50" H 8450 3000 50  0001 C CNN
+F 0 "#PWR053" H 8450 3000 50  0001 C CNN
 F 1 "+3V3" H 8450 3290 50  0000 C CNN
 F 2 "" H 8450 3150 60  0000 C CNN
@@
 Wire Wire Line
 	8150 3150 8450 3150
+Text GLabel 6750 3800 0    60   Input ~ 0
+A16
+Wire Wire Line
+	6400 4825 6400 5050
 $EndSCHEMATC

Commit message: Stab at full PCB
replace DIP36 128KB RAM with TSOP44 512KB RAM
change footprints for many components to SMD
sample PCB layout
Parts:
- removed U9: KM681000BLP-7, Housings_DIP:DIP-32_W15.24mm, symbol KM681000BLP-7
- added C18: 0.1 µF, Capacitors_SMD:C_0805, symbol C
- added U7: 71V424S15PHGI8, TSOP44-II:TSOP44-II, symbol 71V424S15PHGI8
- C16: renamed from C4; footprint Capacitors_ThroughHole:C_Disc_D6_P5 -> Capacitors_SMD:C_0805
- C17: renamed from C5; footprint Capacitors_ThroughHole:C_Disc_D6_P5 -> Capacitors_SMD:C_0805
- R11: renamed from R9; footprint Resistors_ThroughHole:Resistor_Horizontal_RM10mm -> Resistors_SMD:R_0805
- R12: renamed from R10; footprint Resistors_ThroughHole:Resistor_Horizontal_RM10mm -> Resistors_SMD:R_0805
- R13: renamed from R16; footprint Resistors_ThroughHole:Resistor_Horizontal_RM10mm -> Resistors_SMD:R_0805
- U6: renamed from U8; footprint Housings_DIP:DIP-40_W15.24mm -> Housings_QFP:LQFP-44_10x10mm_Pitch0.8mm
Connections:
- wire segments 55 -> 56
Other:
- moved on the sheet: C17
