File: alice3/kicad/MOBO_SMD/VIDEO.sch (KiCad schematic (older format))
At the start: 11 parts, among them P1 CONN_01X05, SW1 RESET, U2 VGA_daughter_board, U3 Propeller_P8X32A-D40, U4 24LC256, U5 Propeller_Plug, Y1 5 MHz

Commit message: Stab at full PCB
replace DIP36 128KB RAM with TSOP44 512KB RAM
change footprints for many components to SMD
sample PCB layout
Parts:
- C1: renamed from C2; footprint Capacitors_ThroughHole:C_Disc_D6_P5 -> Capacitors_SMD:C_0805
- D1: renamed from D2; footprint LEDs:LED-5MM -> LEDs:LED_0805
- R1: renamed from R2; footprint Resistors_ThroughHole:Resistor_Horizontal_RM10mm -> Resistors_SMD:R_0805
- R2: renamed from R3; footprint Resistors_ThroughHole:Resistor_Horizontal_RM10mm -> Resistors_SMD:R_0805
- U2: renamed from U3; footprint Housings_DIP:DIP-40_W15.24mm -> Housings_QFP:LQFP-44_10x10mm_Pitch0.8mm
- renumbered U2 to U1, U4 to U3, U5 to U4
Changed lines of the file:
@@
 LIBS:regul
 LIBS:ldo
+LIBS:71v424s15phgi8
 LIBS:MOBO_SMD-cache
 EELAYER 25 0
@@
 $EndDescr
 $Comp
-L Propeller_P8X32A-D40 U3
+L Propeller_P8X32A-D40 U2
 U 1 1 566E498F
 P 6800 3400
-F 0 "U3" H 6500 4700 60  0000 C CNN
+F 0 "U2" H 6500 4700 60  0000 C CNN
 F 1 "Propeller_P8X32A-D40" H 6800 2100 60  0000 C CNN
-F 2 "Housings_DIP:DIP-40_W15.24mm" H 6800 3200 60  0001 C CNN
+F 2 "Housings_QFP:LQFP-44_10x10mm_Pitch0.8mm" H 6800 3200 60  0001 C CNN
 F 3 "" H 6800 3200 60  0000 C CNN
 	1    6800 3400
@@
 $EndComp
 $Comp
-L VGA_daughter_board U2
+L VGA_daughter_board U1
 U 1 1 5681E1A9
 P 5000 4150
-F 0 "U2" H 4750 4950 60  0000 C CNN
+F 0 "U1" H 4750 4950 60  0000 C CNN
 F 1 "VGA_daughter_board" H 5000 3300 60  0000 C CNN
 F 2 "Pin_Headers:Pin_Header_Straight_1x14" H 5000 4200 60  0001 C CNN
@@
 $EndComp
 $Comp
-L 24LC256 U4
+L 24LC256 U3
 U 1 1 5681F117
 P 8900 4150
-F 0 "U4" H 8650 4450 60  0000 C CNN
+F 0 "U3" H 8650 4450 60  0000 C CNN
 F 1 "24LC256" H 8800 3850 60  0000 C CNN
 F 2 "Housings_DIP:DIP-8_W7.62mm" H 8900 4050 60  0001 C CNN
@@
 $EndComp
 $Comp
-L R R3
+L R R2
 U 1 1 5681F454
 P 8100 3800
-F 0 "R3" V 8180 3800 50  0000 C CNN
+F 0 "R2" V 8180 3800 50  0000 C CNN
 F 1 "10k" V 8100 3800 50  0000 C CNN
-F 2 "Resistors_ThroughHole:Resistor_Horizontal_RM10mm" V 8030 3800 50  0001 C CNN
+F 2 "Resistors_SMD:R_0805" V 8030 3800 50  0001 C CNN
 F 3 "" H 8100 3800 50  0000 C CNN
 	1    8100 3800
@@
 $EndComp
 $Comp
-L Propeller_Plug U5
+L Propeller_Plug U4
 U 1 1 5681F4AC
 P 9600 2850
-F 0 "U5" H 9500 3150 60  0000 C CNN
+F 0 "U4" H 9500 3150 60  0000 C CNN
 F 1 "Propeller_Plug" H 9650 2500 60  0000 C CNN
 F 2 "Pin_Headers:Pin_Header_Angled_1x04" H 9600 2850 60  0001 C CNN
@@
 $EndComp
 $Comp
-L LED D2
+L LED D1
 U 1 1 56821EAA
 P 5700 2600
-F 0 "D2" H 5700 2700 50  0000 C CNN
+F 0 "D1" H 5700 2700 50  0000 C CNN
 F 1 "DEBUG" H 5700 2500 50  0000 C CNN
-F 2 "LEDs:LED-5MM" H 5700 2600 50  0001 C CNN
+F 2 "LEDs:LED_0805" H 5700 2600 50  0001 C CNN
 F 3 "" H 5700 2600 50  0000 C CNN
 	1    5700 2600
@@
 $EndComp
 $Comp
-L R R2
+L R R1
 U 1 1 56821F00
 P 5250 2600
-F 0 "R2" V 5330 2600 50  0000 C CNN
+F 0 "R1" V 5330 2600 50  0000 C CNN
 F 1 "100" V 5250 2600 50  0000 C CNN
-F 2 "Resistors_ThroughHole:Resistor_Horizontal_RM10mm" V 5180 2600 50  0001 C CNN
+F 2 "Resistors_SMD:R_0805" V 5180 2600 50  0001 C CNN
 F 3 "" H 5250 2600 50  0000 C CNN
 	1    5250 2600
@@
 /RD
 $Comp
-L C C2
+L C C1
 U 1 1 568DD525
 P 5800 1950
-F 0 "C2" H 5825 2050 50  0000 L CNN
+F 0 "C1" H 5825 2050 50  0000 L CNN
 F 1 "0.1 µF" H 5825 1850 50  0000 L CNN
-F 2 "Capacitors_ThroughHole:C_Disc_D6_P5" H 5838 1800 50  0001 C CNN
+F 2 "Capacitors_SMD:C_0805" H 5838 1800 50  0001 C CNN
 F 3 "" H 5800 1950 50  0000 C CNN
 	1    5800 1950

Commit message: switch Propeller ROM to SOIC8
Parts:
- U3: footprint Housings_DIP:DIP-8_W7.62mm -> Housings_SOIC:SOIC-8_3.9x4.9mm_Pitch1.27mm
Changed lines of the file:
@@
 F 0 "U3" H 8650 4450 60  0000 C CNN
 F 1 "24LC256" H 8800 3850 60  0000 C CNN
-F 2 "Housings_DIP:DIP-8_W7.62mm" H 8900 4050 60  0001 C CNN
+F 2 "Housings_SOIC:SOIC-8_3.9x4.9mm_Pitch1.27mm" H 8900 4050 60  0001 C CNN
 F 3 "" H 8900 4050 60  0000 C CNN
 	1    8900 4150

Commit message: set crystals to SMD footprints
Parts:
- Y1: footprint Crystals:Crystal_HC50-U_Vertical -> Crystals:Crystal_HC49-SD_SMD
Changed lines of the file:
@@
 F 0 "Y1" H 7750 4600 50  0000 C CNN
 F 1 "5 MHz" H 7750 4300 50  0000 C CNN
-F 2 "Crystals:Crystal_HC50-U_Vertical" H 7750 4450 50  0001 C CNN
+F 2 "Crystals:Crystal_HC49-SD_SMD" H 7750 4450 50  0001 C CNN
 F 3 "" H 7750 4450 50  0000 C CNN
 	1    7750 4450

Commit message: interpolate VGA and PS/2 from Parallax board
Parts:
- removed U1: VGA_daughter_board, Pin_Headers:Pin_Header_Straight_1x14, symbol VGA_daughter_board
- added J?: VGA, symbol VGA
- added R? (x5): 240, symbol R
- added R? (x3): 470, symbol R
Connections:
- net labels added: VGA_B0, VGA_B1, VGA_G0, VGA_G1, VGA_HSYNC, VGA_R0, VGA_R1, VGA_VSYNC
- net labels removed: KBD_CLK, KBD_DATA
- wire segments 94 -> 134
- no-connect marks 2 -> 4
Other:
- moved on the sheet: C1, D1, P1, R1, R2, SW1, U3, U4, Y1
