File: alice3/kicad/MOBO_SMD/VIDEO.sch (KiCad schematic (older format))
At the start: 17 parts, among them J1 VGA, P1 CONN_01X05, SW1 RESET, U2 Propeller_P8X32A-Q44, U3 24LC256, U4 Propeller_Plug, Y1 5 MHz

Commit message: Assign parts to footprints.
Parts:
- R14, R15, R16, R17, R18, R19, R20, R21: footprint (none) -> Resistors_SMD:R_0805
- U2: footprint (none) -> Housings_QFP:LQFP-44_10x10mm_Pitch0.8mm
Changed lines of the file:
@@
 $EndDescr
 $Comp
-L GND #PWR7
+L GND #PWR01
 U 1 1 566E4A0D
 P 3700 3900
-F 0 "#PWR7" H 3700 3650 50  0001 C CNN
+F 0 "#PWR01" H 3700 3650 50  0001 C CNN
 F 1 "GND" H 3700 3750 50  0000 C CNN
 F 2 "" H 3700 3900 50  0000 C CNN
@@
 $EndComp
 $Comp
-L +3.3V #PWR6
+L +3.3V #PWR02
 U 1 1 566E4A37
 P 3700 900
-F 0 "#PWR6" H 3700 750 50  0001 C CNN
+F 0 "#PWR02" H 3700 750 50  0001 C CNN
 F 1 "+3.3V" H 3700 1040 50  0000 C CNN
 F 2 "" H 3700 900 50  0000 C CNN
@@
 $EndComp
 $Comp
-L GND #PWR11
+L GND #PWR03
 U 1 1 566E4C07
 P 6250 1550
-F 0 "#PWR11" H 6250 1300 50  0001 C CNN
+F 0 "#PWR03" H 6250 1300 50  0001 C CNN
 F 1 "GND" H 6250 1400 50  0000 C CNN
 F 2 "" H 6250 1550 50  0000 C CNN
@@
 $EndComp
 $Comp
-L GND #PWR10
+L GND #PWR04
 U 1 1 5681F164
 P 5950 3550
-F 0 "#PWR10" H 5950 3300 50  0001 C CNN
+F 0 "#PWR04" H 5950 3300 50  0001 C CNN
 F 1 "GND" H 5950 3400 50  0000 C CNN
 F 2 "" H 5950 3550 50  0000 C CNN
@@
 $EndComp
 $Comp
-L +3.3V #PWR12
+L +3.3V #PWR05
 U 1 1 5681F2C2
 P 7050 3000
-F 0 "#PWR12" H 7050 2850 50  0001 C CNN
+F 0 "#PWR05" H 7050 2850 50  0001 C CNN
 F 1 "+3.3V" H 7050 3140 50  0000 C CNN
 F 2 "" H 7050 3000 50  0000 C CNN
@@
 $EndComp
 $Comp
-L GND #PWR13
+L GND #PWR06
 U 1 1 5681F2E8
 P 7300 3300
-F 0 "#PWR13" H 7300 3050 50  0001 C CNN
+F 0 "#PWR06" H 7300 3050 50  0001 C CNN
 F 1 "GND" H 7300 3150 50  0000 C CNN
 F 2 "" H 7300 3300 50  0000 C CNN
@@
 $EndComp
 $Comp
-L +3.3V #PWR9
+L +3.3V #PWR07
 U 1 1 5681F435
 P 5700 2750
-F 0 "#PWR9" H 5700 2600 50  0001 C CNN
+F 0 "#PWR07" H 5700 2600 50  0001 C CNN
 F 1 "+3.3V" H 5700 2890 50  0000 C CNN
 F 2 "" H 5700 2750 50  0000 C CNN
@@
 $EndComp
 $Comp
-L GND #PWR8
+L GND #PWR08
 U 1 1 56826035
 P 5050 1550
-F 0 "#PWR8" H 5050 1300 50  0001 C CNN
+F 0 "#PWR08" H 5050 1300 50  0001 C CNN
 F 1 "GND" H 5050 1400 50  0000 C CNN
 F 2 "" H 5050 1550 50  0000 C CNN
@@
 $EndComp
 $Comp
-L GND #PWR5
+L GND #PWR09
 U 1 1 568DD571
 P 3400 1400
-F 0 "#PWR5" H 3400 1150 50  0001 C CNN
+F 0 "#PWR09" H 3400 1150 50  0001 C CNN
 F 1 "GND" H 3400 1250 50  0000 C CNN
 F 2 "" H 3400 1400 50  0000 C CNN
@@
 $EndComp
 $Comp
-L GND #PWR1
+L GND #PWR010
 U 1 1 56A0506B
 P 1000 3050
-F 0 "#PWR1" H 1000 2800 50  0001 C CNN
+F 0 "#PWR010" H 1000 2800 50  0001 C CNN
 F 1 "GND" H 1000 2900 50  0000 C CNN
 F 2 "" H 1000 3050 50  0000 C CNN
@@
 $EndComp
 $Comp
-L +3.3V #PWR2
+L +3.3V #PWR011
 U 1 1 56A050A3
 P 1300 3050
-F 0 "#PWR2" H 1300 2900 50  0001 C CNN
+F 0 "#PWR011" H 1300 2900 50  0001 C CNN
 F 1 "+3.3V" H 1300 3190 50  0000 C CNN
 F 2 "" H 1300 3050 50  0000 C CNN
@@
 F 0 "J1" H 3800 6975 60  0000 C CNN
 F 1 "VGA" H 4050 5425 60  0000 C CNN
-F 2 "" H 4050 6175 60  0000 C CNN
+F 2 "" H 4050 6175 60  0001 C CNN
 F 3 "" H 4050 6175 60  0000 C CNN
 	1    4050 6175
@@
 $EndComp
 $Comp
-L GND #PWR4
+L GND #PWR012
 U 1 1 56CDE065
 P 3325 6775
-F 0 "#PWR4" H 3325 6525 50  0001 C CNN
+F 0 "#PWR012" H 3325 6525 50  0001 C CNN
 F 1 "GND" H 3325 6625 50  0000 C CNN
 F 2 "" H 3325 6775 60  0000 C CNN
@@
 Connection ~ 3325 6625
 $Comp
-L +5V #PWR3
+L +5V #PWR013
 U 1 1 56CDE22E
 P 3125 5600
-F 0 "#PWR3" H 3125 5450 50  0001 C CNN
+F 0 "#PWR013" H 3125 5450 50  0001 C CNN
 F 1 "+5V" H 3125 5740 50  0000 C CNN
 F 2 "" H 3125 5600 60  0000 C CNN
@@
 F 0 "R20" V 5130 5925 50  0000 C CNN
 F 1 "240" V 5050 5925 50  0000 C CNN
-F 2 "" V 4980 5925 30  0000 C CNN
+F 2 "Resistors_SMD:R_0805" V 4980 5925 30  0001 C CNN
 F 3 "" H 5050 5925 30  0000 C CNN
 	1    5050 5925
@@
 F 0 "R21" V 5130 6125 50  0000 C CNN
 F 1 "240" V 5050 6125 50  0000 C CNN
-F 2 "" V 4980 6125 30  0000 C CNN
+F 2 "Resistors_SMD:R_0805" V 4980 6125 30  0001 C CNN
 F 3 "" H 5050 6125 30  0000 C CNN
 	1    5050 6125
@@
 F 0 "R18" V 1730 6575 50  0000 C CNN
 F 1 "240" V 1650 6575 50  0000 C CNN
-F 2 "" V 1580 6575 30  0000 C CNN
+F 2 "Resistors_SMD:R_0805" V 1580 6575 30  0001 C CNN
 F 3 "" H 1650 6575 30  0000 C CNN
 	1    1650 6575
@@
 F 0 "R19" V 1730 6750 50  0000 C CNN
 F 1 "470" V 1650 6750 50  0000 C CNN
-F 2 "" V 1580 6750 30  0000 C CNN
+F 2 "Resistors_SMD:R_0805" V 1580 6750 30  0001 C CNN
 F 3 "" H 1650 6750 30  0000 C CNN
 	1    1650 6750
@@
 F 0 "R16" V 1730 6225 50  0000 C CNN
 F 1 "240" V 1650 6225 50  0000 C CNN
-F 2 "" V 1580 6225 30  0000 C CNN
+F 2 "Resistors_SMD:R_0805" V 1580 6225 30  0001 C CNN
 F 3 "" H 1650 6225 30  0000 C CNN
 	1    1650 6225
@@
 F 0 "R17" V 1730 6400 50  0000 C CNN
 F 1 "470" V 1650 6400 50  0000 C CNN
-F 2 "" V 1580 6400 30  0000 C CNN
+F 2 "Resistors_SMD:R_0805" V 1580 6400 30  0001 C CNN
 F 3 "" H 1650 6400 30  0000 C CNN
 	1    1650 6400
@@
 F 0 "R14" V 1730 5875 50  0000 C CNN
 F 1 "240" V 1650 5875 50  0000 C CNN
-F 2 "" V 1580 5875 30  0000 C CNN
+F 2 "Resistors_SMD:R_0805" V 1580 5875 30  0001 C CNN
 F 3 "" H 1650 5875 30  0000 C CNN
 	1    1650 5875
@@
 F 0 "R15" V 1730 6050 50  0000 C CNN
 F 1 "470" V 1650 6050 50  0000 C CNN
-F 2 "" V 1580 6050 30  0000 C CNN
+F 2 "Resistors_SMD:R_0805" V 1580 6050 30  0001 C CNN
 F 3 "" H 1650 6050 30  0000 C CNN
 	1    1650 6050
@@
 F 0 "U2" H 4100 4050 60  0000 C CNN
 F 1 "Propeller_P8X32A-Q44" H 4450 1050 60  0000 C CNN
-F 2 "" H 4400 2350 60  0000 C CNN
+F 2 "Housings_QFP:LQFP-44_10x10mm_Pitch0.8mm" H 4400 2350 60  0001 C CNN
 F 3 "" H 4400 2350 60  0000 C CNN
 	1    4400 2550
