File: alice3/kicad/MOBO_SMD/MOBO_SMD.kicad_pcb (KiCad board)
At the start: 2 copper layers, 90.2 x 48.3 mm, 67 parts, among them CON1 MicroSD, J1 VGA, P1 CONN_01X05, P2 USB_OTG, P3 UART1, SW1 RESET, SW2 SOFT RESET, U1 Z80CPU-SMD, U2 Propeller_P8X32A-Q44, U3 24LC256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

Commit message: More routing.
Parts:
- CON1: footprint microsd:microsd_socket -> Molex:microsd_1040310811
- moved CON1 7.87 mm to (124.2, 75.2), turned to 180 degrees
Routing:
- net VGA_R0: track 0.00 -> 50.3 mm, vias 0 -> 2
- net VGA_R1: track 0.00 -> 48.6 mm, vias 0 -> 2
- net VGA_G1: track 0.00 -> 43.5 mm, vias 0 -> 2
- net VGA_G0: track 0.00 -> 41.1 mm, vias 0 -> 2
- net VGA_B1: track 0.00 -> 37.7 mm, vias 0 -> 2
- net VGA_B0: track 0.00 -> 35.8 mm, vias 0 -> 2

Commit message: More routing.
Routing:
- net A1: track 21.3 -> 96.5 mm, vias 2 -> 8
- net D1: track 21.0 -> 85.4 mm, vias 0 -> 3
- net A17: track 0.00 -> 61.8 mm, vias 0 -> 6
- net A7: track 19.5 -> 72.4 mm, vias 2 -> 5
- net D4: track 53.3 -> 105.1 mm, vias 2 -> 3
- net D5: track 56.3 -> 102.8 mm, vias 2 -> 3
- net D6: track 58.4 -> 103.6 mm, vias 2 -> 3
- net A3: track 27.4 -> 69.2 mm, vias 2 -> 8
- net A0: track 43.5 -> 79.6 mm, vias 8 -> 10
- net A10: track 29.4 -> 61.5 mm, vias 2 -> 3
- net A2: track 60.1 -> 88.0 mm, vias 6 -> 7
- net VGA_HSYNC: track 3.87 -> 20.0 mm, vias 2 -> 0
- net VGA_VSYNC: track 21.1 -> 24.4 mm
- net A12: track 52.2 -> 54.6 mm
- net A16: track 57.4 -> 59.8 mm
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
Commit message: More routing.
Routing:
- net CLK: track 0.00 -> 50.0 mm, vias 0 -> 2
- net /IORQ: track 26.5 -> 75.8 mm, vias 2 -> 3
- net D2: track 57.2 -> 95.8 mm, vias 2 -> 3
- net D3: track 62.4 -> 99.9 mm, vias 4 -> 5
- net D7: track 63.5 -> 100.7 mm, vias 2 -> 3
- net A1: track 96.5 -> 85.3 mm
- net /BUSRQ: track 29.2 -> 30.8 mm
- net /HALT: track 29.2 -> 30.6 mm
- net /WR: track 48.8 -> 47.5 mm
- net A14: track 54.8 -> 55.9 mm
- net A11: track 41.8 -> 40.7 mm
- net A0: track 79.6 -> 78.5 mm
- net +3V3: track 186.9 -> 188.0 mm
- net A5: track 46.5 -> 45.5 mm
- net D0: track 86.6 -> 85.7 mm
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
Commit message: More routing.
Routing:
- net +3V3: track 188.0 -> 275.2 mm
- net A16: track 59.9 -> 0.00 mm, vias 2 -> 0
- net /RESET: track 0.00 -> 57.3 mm, vias 0 -> 4
- net GND: track 376.3 -> 426.4 mm, vias 22 -> 25
- net Net-(R1-Pad1): track 0.00 -> 44.7 mm, vias 0 -> 5
- net /IO/SCK: track 26.9 -> 47.9 mm, vias 2 -> 4
- net /IO/DI: track 27.9 -> 48.8 mm
- net /IO/DO: track 20.5 -> 40.6 mm, vias 2 -> 4
- net /IO/CS: track 0.00 -> 19.3 mm
- net D0: track 85.7 -> 68.2 mm
- net Net-(JP1-Pad2): track 8.95 -> 21.4 mm, vias 0 -> 2
- net Net-(SW2-Pad1): track 0.00 -> 7.95 mm
- net /WR: track 47.5 -> 46.8 mm

Commit message: More routing.
Parts:
- turned R12 to 270 degrees
Routing:
- net ~PROP_READY~: track 0.00 -> 75.6 mm, vias 0 -> 4
- net Net-(P1-Pad3): track 0.00 -> 57.8 mm, vias 0 -> 1
- net /RESET: track 57.3 -> 114.3 mm, vias 4 -> 9
- net Net-(U2-Pad37): track 0.00 -> 43.5 mm
- net A16: track 0.00 -> 42.4 mm, vias 0 -> 2
- net Net-(U2-Pad38): track 0.00 -> 40.2 mm
- net Net-(SW2-Pad1): track 7.95 -> 43.7 mm, vias 0 -> 4
- net Net-(P1-Pad5): track 0.00 -> 32.5 mm, vias 0 -> 2
- net Net-(P1-Pad4): track 0.00 -> 29.8 mm, vias 0 -> 2
- net +3V3: track 275.2 -> 302.8 mm, vias 2 -> 4
- net D0: track 68.2 -> 93.6 mm, vias 4 -> 6
- net Net-(P3-Pad1): track 0.00 -> 24.0 mm, vias 0 -> 2
- net /IO/CS: track 19.3 -> 42.1 mm, vias 0 -> 4
- net Net-(P3-Pad2): track 0.00 -> 20.6 mm, vias 0 -> 2
- net GND: track 426.4 -> 446.2 mm, vias 25 -> 27
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
Commit message: More routing.
Routing:
- net KBD_DATA: track 0.00 -> 71.3 mm, vias 0 -> 4
- net KBD_CLK: track 0.00 -> 69.1 mm, vias 0 -> 4
- net /RD: track 29.0 -> 82.3 mm, vias 2 -> 7
- net /WR: track 46.8 -> 80.6 mm, vias 2 -> 6
- net +3V3: track 302.8 -> 317.7 mm
- net GND: track 446.2 -> 460.0 mm, vias 27 -> 29
- net A7: track 76.9 -> 79.8 mm
- net D0: track 93.6 -> 95.9 mm
- net /Z80_RESET: track 31.3 -> 29.4 mm
- net A17: track 62.5 -> 61.3 mm
- net D5: track 112.3 -> 113.3 mm
- net /IORQ: track 73.1 -> 72.1 mm
- net D7: track 105.8 -> 106.6 mm
- net A9: track 41.1 -> 40.3 mm
- net A15: track 54.9 -> 55.6 mm
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
Commit message: Done routing.
Routing:
- net USB_ID: track 0.00 -> 92.6 mm, vias 0 -> 4
- net USB_D_N: track 0.00 -> 92.2 mm, vias 0 -> 4
- net USB_D_P: track 0.00 -> 87.2 mm, vias 0 -> 4
- net USB_DET: track 0.00 -> 18.7 mm, vias 0 -> 2
- net +5V: track 96.1 -> 100.4 mm
- net A11: track 41.9 -> 45.7 mm
- net A3: track 70.3 -> 73.9 mm
- net /BUSRQ: track 30.7 -> 33.1 mm
- net GND: track 460.0 -> 462.3 mm
- net A6: track 47.8 -> 49.8 mm
- net A9: track 40.3 -> 42.2 mm
- net A15: track 55.6 -> 57.5 mm
- net A16: track 42.7 -> 44.5 mm
- net ~PROP_READY~: track 76.1 -> 77.7 mm
- net A0: track 78.8 -> 80.4 mm
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